File: sdr_kicad/clock_si5351.kicad_sch (KiCad schematic)
At the start: 9 parts, among them Y2 25MHz

Commit message: Add Python KiCad helper library and JLCPCB component libraries
- Add kicad_lib: Python library for parsing, creating, and validating KiCad files
  - S-expression parser and writer for .kicad_sym and .kicad_sch files
  - Immutable dataclasses for symbols, schematics, pins, wires, etc.
  - SymbolBuilder with fluent API for programmatic symbol creation
  - ERC validation runner with configurable rules
  - Result type for explicit error handling

- Add custom_lib: JLCPCB component libraries downloaded via JLC2KiCadLib
  - 21 symbol definitions (.kicad_sym)
  - 19 footprints with 3D STEP models
  - Includes STM32G474, TPS25750D, BQ25798, Si5351A, FT4232HL, etc.

- Update CLAUDE.md with kicad_lib documentation and usage examples

- Update schematic sheets with embedded lib_symbols and wiring
Parts:
- removed C40, C41: 10pF, Capacitor_SMD:C_0402_1005Metric, symbol Device:C
- removed C42, C44: 100nF, Capacitor_SMD:C_0402_1005Metric, symbol Device:C
- removed C43: 10uF, Capacitor_SMD:C_0603_1608Metric, symbol Device:C
- removed R50, R51, R52: 47R, Resistor_SMD:R_0402_1005Metric, symbol Device:R
- removed Y2: 25MHz, Crystal:Crystal_HC49-4H_Vertical, symbol Device:Crystal
- added C15: 100n, Capacitor_SMD:C_0402_1005Metric, symbol Device:C
- added D1, D2: 1N4148, Diode_SMD:D_SOD-323, symbol Device:D
- added R4, R5: 1k, Resistor_SMD:R_0402_1005Metric, symbol Device:R
- added U3: Si5351A-B-GT, Package_SO:MSOP-10_3x3mm_P0.5mm, symbol SI5351A:SI5351A-B-GT
- added Y1: 27MHz, Crystal:Crystal_HC49-4H_Vertical, symbol Device:Crystal
Connections:
- net +3V3: now also R4.1, R5.1, U3.1 (VDD)
- net +5V: now also D1.1 (K)
- net CLK0: now also U3.10 (CLK0)
- net CLK1: now also U3.9 (CLK1)
- net CLK2: now also U3.6 (CLK2)
- new net: C15.1, U3.7 (VDDO)
- new net: D1.2 (A), D2.1 (K)
- new net: U3.2 (XA), Y1.2
- new net: U3.3 (XB), Y1.1
- new net GND: C15.2, U3.8 (GND)
- new net PC4_SDA: R5.2, U3.5 (SDA)
- new net PC5_SCL: R4.2, U3.4 (SCL)
Other:
- note added: "Si5351A Clock Generator I2C Address: 0x60 27MHz Crystal Reference"
- note removed: "25MHz Reference Crystal"
- note removed: "Clock Output Conditioning"
- note removed: "Power Decoupling"
- note removed: "Si5351 outputs are CMOS push-pull. For driving FST3253 QSD switches: • Direct connection OK at 3.3V • Series resistor (33-100Ω) for impedance matching and EMI • AC coupling if DC offset needed Output Series Resistors: R50, R51, R52: 47Ω 0402 LCSC: C25118 (Basic)"
- note removed: "Si5351A Features: • 8 Independent Outputs (A variant) • 8kHz - 160MHz output range • I2C Interface (Addr: 0x60) • Dual PLLs for phase control • <1 Hz frequency resolution • Low jitter (<1ps RMS) LCSC Part: C506891 Package: MSOP-10 Clock Outputs Used: • CLK0: I-channel LO (0°) • CLK1: Q-channel LO (90°) • CLK2: TX carrier / BFO Quadrature Generation: PLL phase offset method: CLK1 phase = CLK0 + 90°"
- note removed: "Si5351A-B-GT Clock Synthesizer"
- note removed: "VDD (3.3V Core): • 100nF ceramic close to pin • 10uF bulk nearby VDDO (Output driver, 3.3V or 5V): • 100nF ceramic close to pin • Can run at 5V for higher drive Note: Keep VDD and VDDO decoupling separate for best noise performance."
