File: sdr_kicad/clock_si5351.kicad_sch (KiCad schematic)
At the start: 7 parts, among them U3 Si5351A-B-GT, Y1 27MHz

Commit message: add firmware and readme
Connections:
- net at C15.1, U3.7 (VDDO): now also D2.2 (A)
Other:
- note added: "Si5351A Clock Generator I2C Address: 0x60 27MHz Crystal Reference VDDO Protection: +5V clamp via D1/D2 series to +3V3 rail"
- note removed: "Si5351A Clock Generator I2C Address: 0x60 27MHz Crystal Reference"
- moved on the sheet: C15, D1, D2
