File: sdr_kicad/rf_section.kicad_sch (KiCad schematic)
At the start: 8 parts, among them Q1 2N7002

Commit message: Add missing schematic symbols and fix hierarchical connections
- Add USB-C receptacles (J1, J2) and USBLC6-2SC6 ESD ICs to usb_connectors
- Add FST3253 QSD, EC2-3SNU relays (K1-K5), SMA connector, 1N5711 diodes to rf_section
- Add missing sheet pins for proper hierarchical signal routing
- Remove invalid comment lines that broke KiCad parser
- Update power management to TPS25750D/BQ25798 architecture for 4S battery support
- ERC reduced from 89 to 82 violations (remaining are unwired connections)
Parts:
- added D1, D2: 1N5711, Diode_SMD:D_SOD-323, symbol Diode:1N5711
- added J10: SMA, Connector_Coaxial:SMA_Amphenol_132289_EdgeMount, symbol Connector:Conn_Coaxial
- added K1, K2, K3, K4, K5: EC2-3SNU, Relay_SMD:Relay_DPDT_Kemet_EC2, symbol Relay:EC2-3SNU
- added U20: FST3253, Package_SO:TSSOP-16_4.4x5mm_P0.65mm, symbol Analog_Switch:FST3253
Changed lines of the file:
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@@
+    )
+  )
+  (symbol
+    (lib_id "Analog_Switch:FST3253")
+    (at 241.3 127 0)
+    (unit 1)
+    (exclude_from_sim no)
+    (in_bom yes)
+    (on_board yes)
+    (dnp no)
+    (uuid "u-qsd")
+    (property "Reference" "U20"
+      (at 241.3 106.68 0)
+      (effects (font (size 1.27 1.27)))
+    )
+    (property "Value" "FST3253"
+      (at 241.3 109.22 0)
+      (effects (font (size 1.27 1.27)))
+    )
+    (property "Footprint" "Package_SO:TSSOP-16_4.4x5mm_P0.65mm"
+      (at 241.3 127 0)
+      (effects (font (size 1.27 1.27)) hide)
+    )
+    (property "LCSC" "C55736"
+      (at 241.3 127 0)
+      (effects (font (size 1.27 1.27)) hide)
+    )
+  )
+  (symbol
+    (lib_id "Relay:EC2-3SNU")
+    (at 101.6 127 0)
+    (unit 1)
+    (exclude_from_sim no)
+    (in_bom yes)
+    (on_board yes)
+    (dnp no)
+    (uuid "k1-relay80m")
+    (property "Reference" "K1"
+      (at 101.6 111.76 0)
+      (effects (font (size 1.27 1.27)))
+    )
+    (property "Value" "EC2-3SNU"
+      (at 101.6 114.3 0)
+      (effects (font (size 1.27 1.27)))
+    )
+    (property "Footprint" "Relay_SMD:Relay_DPDT_Kemet_EC2"
+      (at 101.6 127 0)
+      (effects (font (size 1.27 1.27)) hide)
+    )
+    (property "LCSC" "C132490"
+      (at 101.6 127 0)
+      (effects (font (size 1.27 1.27)) hide)
+    )
+  )
+  (symbol
+    (lib_id "Relay:EC2-3SNU")
+    (at 101.6 157.48 0)
+    (unit 1)
+    (exclude_from_sim no)
+    (in_bom yes)
+    (on_board yes)
+    (dnp no)
+    (uuid "k2-relay40m")
+    (property "Reference" "K2"
+      (at 101.6 142.24 0)
+      (effects (font (size 1.27 1.27)))
+    )
+    (property "Value" "EC2-3SNU"
+      (at 101.6 144.78 0)
+      (effects (font (size 1.27 1.27)))
+    )
+    (property "Footprint" "Relay_SMD:Relay_DPDT_Kemet_EC2"
+      (at 101.6 157.48 0)
+      (effects (font (size 1.27 1.27)) hide)
+    )
+    (property "LCSC" "C132490"
+      (at 101.6 157.48 0)
+      (effects (font (size 1.27 1.27)) hide)
+    )
+  )
+  (symbol
+    (lib_id "Relay:EC2-3SNU")
+    (at 101.6 187.96 0)
+    (unit 1)
+    (exclude_from_sim no)
+    (in_bom yes)
+    (on_board yes)
+    (dnp no)
+    (uuid "k3-relay20m")
+    (property "Reference" "K3"
+      (at 101.6 172.72 0)
+      (effects (font (size 1.27 1.27)))
+    )
+    (property "Value" "EC2-3SNU"
+      (at 101.6 175.26 0)
+      (effects (font (size 1.27 1.27)))
+    )
+    (property "Footprint" "Relay_SMD:Relay_DPDT_Kemet_EC2"
+      (at 101.6 187.96 0)
+      (effects (font (size 1.27 1.27)) hide)
+    )
+    (property "LCSC" "C132490"
+      (at 101.6 187.96 0)
+      (effects (font (size 1.27 1.27)) hide)
+    )
+  )
+  (symbol
+    (lib_id "Relay:EC2-3SNU")
+    (at 101.6 218.44 0)
+    (unit 1)
+    (exclude_from_sim no)
+    (in_bom yes)
+    (on_board yes)
+    (dnp no)
+    (uuid "k4-relay15m")
+    (property "Reference" "K4"
+      (at 101.6 203.2 0)
+      (effects (font (size 1.27 1.27)))
+    )
+    (property "Value" "EC2-3SNU"
+      (at 101.6 205.74 0)
+      (effects (font (size 1.27 1.27)))
+    )
+    (property "Footprint" "Relay_SMD:Relay_DPDT_Kemet_EC2"
+      (at 101.6 218.44 0)
+      (effects (font (size 1.27 1.27)) hide)
+    )
+    (property "LCSC" "C132490"
+      (at 101.6 218.44 0)
+      (effects (font (size 1.27 1.27)) hide)
+    )
+  )
+  (symbol
+    (lib_id "Relay:EC2-3SNU")
+    (at 101.6 248.92 0)
+    (unit 1)
+    (exclude_from_sim no)
+    (in_bom yes)
+    (on_board yes)
+    (dnp no)
+    (uuid "k5-relay10m")
+    (property "Reference" "K5"
+      (at 101.6 233.68 0)
+      (effects (font (size 1.27 1.27)))
+    )
+    (property "Value" "EC2-3SNU"
+      (at 101.6 236.22 0)
+      (effects (font (size 1.27 1.27)))
+    )
+    (property "Footprint" "Relay_SMD:Relay_DPDT_Kemet_EC2"
+      (at 101.6 248.92 0)
+      (effects (font (size 1.27 1.27)) hide)
+    )
+    (property "LCSC" "C132490"
+      (at 101.6 248.92 0)
+      (effects (font (size 1.27 1.27)) hide)
+    )
+  )
+  (symbol
+    (lib_id "Connector:Conn_Coaxial")
+    (at 355.6 50.8 0)
+    (unit 1)
+    (exclude_from_sim no)
+    (in_bom yes)
+    (on_board yes)
+    (dnp no)
+    (uuid "j-ant")
+    (property "Reference" "J10"
+      (at 358.14 45.72 0)
+      (effects (font (size 1.27 1.27)) (justify left))
+    )
+    (property "Value" "SMA"
+      (at 358.14 48.26 0)
+      (effects (font (size 1.27 1.27)) (justify left))
+    )
+    (property "Footprint" "Connector_Coaxial:SMA_Amphenol_132289_EdgeMount"
+      (at 355.6 50.8 0)
+      (effects (font (size 1.27 1.27)) hide)
+    )
+    (property "LCSC" "C496549"
+      (at 355.6 50.8 0)
+      (effects (font (size 1.27 1.27)) hide)
+    )
+  )
+  (symbol
+    (lib_id "Diode:1N5711")
+    (at 279.4 63.5 90)
+    (unit 1)
+    (exclude_from_sim no)
+    (in_bom yes)
+    (on_board yes)
+    (dnp no)
+    (uuid "d1-swr-fwd")
+    (property "Reference" "D1"
+      (at 281.94 60.96 90)
+      (effects (font (size 1.27 1.27)) (justify left))
+    )
+    (property "Value" "1N5711"
+      (at 281.94 63.5 90)
+      (effects (font (size 1.27 1.27)) (justify left))
+    )
+    (property "Footprint" "Diode_SMD:D_SOD-323"
+      (at 279.4 63.5 0)
+      (effects (font (size 1.27 1.27)) hide)
+    )
+    (property "LCSC" "C727110"
+      (at 279.4 63.5 0)
+      (effects (font (size 1.27 1.27)) hide)
+    )
+  )
+  (symbol
+    (lib_id "Diode:1N5711")
+    (at 292.1 63.5 90)
+    (unit 1)
+    (exclude_from_sim no)
+    (in_bom yes)
+    (on_board yes)
+    (dnp no)
+    (uuid "d2-swr-rev")
+    (property "Reference" "D2"
+      (at 294.64 60.96 90)
+      (effects (font (size 1.27 1.27)) (justify left))
+    )
+    (property "Value" "1N5711"
+      (at 294.64 63.5 90)
+      (effects (font (size 1.27 1.27)) (justify left))
+    )
+    (property "Footprint" "Diode_SMD:D_SOD-323"
+      (at 292.1 63.5 0)
+      (effects (font (size 1.27 1.27)) hide)
+    )
+    (property "LCSC" "C727110"
+      (at 292.1 63.5 0)
+      (effects (font (size 1.27 1.27)) hide)
     )
   )

Commit message: Add Python KiCad helper library and JLCPCB component libraries
- Add kicad_lib: Python library for parsing, creating, and validating KiCad files
  - S-expression parser and writer for .kicad_sym and .kicad_sch files
  - Immutable dataclasses for symbols, schematics, pins, wires, etc.
  - SymbolBuilder with fluent API for programmatic symbol creation
  - ERC validation runner with configurable rules
  - Result type for explicit error handling

- Add custom_lib: JLCPCB component libraries downloaded via JLC2KiCadLib
  - 21 symbol definitions (.kicad_sym)
  - 19 footprints with 3D STEP models
  - Includes STM32G474, TPS25750D, BQ25798, Si5351A, FT4232HL, etc.

- Update CLAUDE.md with kicad_lib documentation and usage examples

- Update schematic sheets with embedded lib_symbols and wiring
Parts:
- K1, K2, K3, K4, K5: footprint Relay_SMD:Relay_DPDT_Kemet_EC2 -> Relay_THT:Relay_DPDT_Omron_G5V-2
- Q1: symbol Transistor_FET:2N7002 -> 2N7002:2N7002
- U20: symbol Analog_Switch:FST3253 -> FST3253MX:FST3253MX
Changed lines of the file:
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@@
   )
   (symbol
-    (lib_id "Transistor_FET:2N7002")
+    (lib_id "2N7002:2N7002")
     (at 152.4 127 0)
     (unit 1)
@@
   )
   (symbol
-    (lib_id "Analog_Switch:FST3253")
+    (lib_id "FST3253MX:FST3253MX")
     (at 241.3 127 0)
     (unit 1)
@@
       (effects (font (size 1.27 1.27)))
     )
-    (property "Footprint" "Relay_SMD:Relay_DPDT_Kemet_EC2"
+    (property "Footprint" "Relay_THT:Relay_DPDT_Omron_G5V-2"
       (at 101.6 127 0)
       (effects (font (size 1.27 1.27)) hide)
@@
       (effects (font (size 1.27 1.27)))
     )
-    (property "Footprint" "Relay_SMD:Relay_DPDT_Kemet_EC2"
+    (property "Footprint" "Relay_THT:Relay_DPDT_Omron_G5V-2"
       (at 101.6 157.48 0)
       (effects (font (size 1.27 1.27)) hide)
@@
       (effects (font (size 1.27 1.27)))
     )
-    (property "Footprint" "Relay_SMD:Relay_DPDT_Kemet_EC2"
+    (property "Footprint" "Relay_THT:Relay_DPDT_Omron_G5V-2"
       (at 101.6 187.96 0)
       (effects (font (size 1.27 1.27)) hide)
@@
       (effects (font (size 1.27 1.27)))
     )
-    (property "Footprint" "Relay_SMD:Relay_DPDT_Kemet_EC2"
+    (property "Footprint" "Relay_THT:Relay_DPDT_Omron_G5V-2"
       (at 101.6 218.44 0)
       (effects (font (size 1.27 1.27)) hide)
@@
       (effects (font (size 1.27 1.27)))
     )
-    (property "Footprint" "Relay_SMD:Relay_DPDT_Kemet_EC2"
+    (property "Footprint" "Relay_THT:Relay_DPDT_Omron_G5V-2"
       (at 101.6 248.92 0)
       (effects (font (size 1.27 1.27)) hide)
@@
     )
   )
+  (wire
+    (pts
+      (xy 25.4 50.8)
+      (xy 88.9 50.8)
+    )
+    (uuid "wire-rf-vsys")
+  )
+  (wire
+    (pts
+      (xy 25.4 63.5)
+      (xy 50.8 63.5)
+    )
+    (uuid "wire-rf-pwm")
+  )
+  (wire
+    (pts
+      (xy 25.4 76.2)
+      (xy 50.8 76.2)
+    )
+    (uuid "wire-rf-band")
+  )
+  (wire
+    (pts
+      (xy 254 127)
+      (xy 279.4 127)
+    )
+    (uuid "wire-rf-clki")
+  )
+  (wire
+    (pts
+      (xy 254 144.78)
+      (xy 279.4 144.78)
+    )
+    (uuid "wire-rf-clkq")
+  )
+  (wire
+    (pts
+      (xy 330.2 50.8)
+      (xy 355.6 50.8)
+    )
+    (uuid "wire-rf-ant")
+  )
+  (wire
+    (pts
+      (xy 297.18 127)
+      (xy 330.2 127)
+    )
+    (uuid "wire-rf-rxi")
+  )
+  (wire
+    (pts
+      (xy 297.18 144.78)
+      (xy 330.2 144.78)
+    )
+    (uuid "wire-rf-rxq")
+  )
+  (wire
+    (pts
+      (xy 25.4 88.9)
+      (xy 50.8 88.9)
+    )
+    (uuid "wire-rf-txen")
+  )
   (hierarchical_label "VSYS"
