File: sdr_kicad/rf_section.kicad_sch (KiCad schematic)
At the start: 17 parts, among them J10 SMA, K1 EC2-3SNU, K2 EC2-3SNU, K3 EC2-3SNU, K4 EC2-3SNU, K5 EC2-3SNU, Q1 2N7002, U20 FST3253

Commit message: add firmware and readme
Connections:
- net CLK_I: no longer R40.1
- net CLK_Q: no longer R41.1
- net RX_I: no longer C40.1, R40.2
- net RX_Q: no longer C41.1, R41.2
- removed net GND: C40.2, C41.2, U20.8 (GND)
- no-connect marks 54 -> 0
