File: sdr_kicad/rf_section_yaml.kicad_sch (KiCad schematic)
At the start: 17 parts, among them J10 SMA, K1 EC2-3SNU, K2 EC2-3SNU, K3 EC2-3SNU, K4 EC2-3SNU, K5 EC2-3SNU, Q1 2N7002, U20 FST3253

Commit message: schematic is still quite borked
Parts:
- C30, C31, C40, C41, Q1, R30, R40, R41: JLC_Basic Yes -> (none)
- K1: value EC2-3SNU -> LPF_80m
- K2: value EC2-3SNU -> LPF_40m
- K3: value EC2-3SNU -> LPF_30m_20m
- K4: value EC2-3SNU -> LPF_17m_15m
- K5: value EC2-3SNU -> T_R_Switch
Connections:
- net GND is gone; now on net VSYS: C40.2, C41.2, U20.8 (GND)
- net RX_Q is gone; now on net RX_I: C41.1, R41.2
- net CLK_I: now also U20.1 (OE1#)
- net CLK_Q: now also U20.15 (OE2#)
- net VSYS: now also C30.1, C30.2, C31.1, C31.2, Q1.1 (G), Q1.2 (S), R30.2, U20.14 (S0), U20.3 (1B4)
- no-connect marks 54 -> 10
Other:
- note removed: "5-Band Low Pass Filter"
- note removed: "FST3253 Tayloe Detector • LCSC: C55736 • Driven by Si5351 CLK0/1 Anti-alias LPF: • R: 10k (C25744) • C: 4.7nF (C1538) • Fc: ~3.4kHz"
- note removed: "H-Bridge Class-E Power Amplifier"
- note removed: "LPF VALUES Band |Cutoff| L1=L3 | L2 |C1=C3 | C2 80m |4.5MHz| 2.4uH |2.9uH |1200pF|1500pF 40m |8MHz | 1.2uH |1.5uH | 680pF| 820pF 30/20m|15MHz | 680nH |820nH | 390pF| 470pF 17/15m|22MHz | 470nH |560nH | 270pF| 330pF 12/10m|30MHz | 330nH |390nH | 180pF| 220pF"
- note removed: "Latching Relay Switching • EC2-3SNU DPDT • 3V coil, 10ms pulse • Zero standby current • LCSC: C132490 Driver: 2N7002 (C8545)"
- note removed: "Quadrature Sampling Detector"
- note removed: "SWR Bridge"
- note removed: "Tandem Match: • FT50-43 toroid • 1T primary, 10T secondary • 1N5711 detectors"
- note removed: "uP9636 H-Bridge Driver • VIN: 2.5V-25V (VSYS) • VCC: 4.5V-13.2V • 60A MOSFETs, 5.5mΩ Discrete Alternative: • 4x Si2302 (C10487) • 2x IR2104 driver"
