File: sdr_kicad/sdr_transceiver.kicad_sch (KiCad schematic)
At the start: 0 parts

Commit message: Add missing schematic symbols and fix hierarchical connections
- Add USB-C receptacles (J1, J2) and USBLC6-2SC6 ESD ICs to usb_connectors
- Add FST3253 QSD, EC2-3SNU relays (K1-K5), SMA connector, 1N5711 diodes to rf_section
- Add missing sheet pins for proper hierarchical signal routing
- Remove invalid comment lines that broke KiCad parser
- Update power management to TPS25750D/BQ25798 architecture for 4S battery support
- ERC reduced from 89 to 82 violations (remaining are unwired connections)
Other:
- sheet Clock_Si5351 ports: added +3V3, +5V; removed none
- sheet Debug_FT4232 ports: added USB2_DM, USB2_DP; removed none
- sheet MCU_STM32G4 ports: added I2C1_SCL, I2C1_SDA, TPS_INT; removed I2C_SCL, I2C_SDA
- sheet Power_Management ports: added CC1, CC2, I2C1_SCL, I2C1_SDA, TPS_INT, VBAT+; removed none
- sheet RF_Section ports: added TX_EN; removed none
- sheet USB_Connectors ports: added VBUS; removed VBUS_OUT
Changed lines of the file:
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@@
     (comment 2 "STM32G4 + USB-C PD + 3S Battery")
   )
-  ;; Power symbols
   (symbol
     (lib_id "power:GND")
@@
     )
   )
-  ;; Title text
   (text "SDR TRANSCEIVER - TOP LEVEL"
     (exclude_from_sim no)
@@
     (uuid "desc-text-1")
   )
-  ;; Sheet: Power Management
   (sheet
     (at 25.4 88.9)
@@
       (uuid "pin-3v3-1")
     )
-  )
-  ;; Sheet: MCU
+    (pin "CC1" bidirectional
+      (at 25.4 93.98 180)
+      (effects
+        (font (size 1.524 1.524))
+        (justify left)
+      )
+      (uuid "pin-pwr-cc1-1")
+    )
+    (pin "CC2" bidirectional
+      (at 25.4 99.06 180)
+      (effects
+        (font (size 1.524 1.524))
+        (justify left)
+      )
+      (uuid "pin-pwr-cc2-1")
+    )
+    (pin "I2C1_SCL" bidirectional
+      (at 25.4 104.14 180)
+      (effects
+        (font (size 1.524 1.524))
+        (justify left)
+      )
+      (uuid "pin-pwr-i2c-scl-1")
+    )
+    (pin "I2C1_SDA" bidirectional
+      (at 25.4 109.22 180)
+      (effects
+        (font (size 1.524 1.524))
+        (justify left)
+      )
+      (uuid "pin-pwr-i2c-sda-1")
+    )
+    (pin "TPS_INT" output
+      (at 76.2 114.3 0)
+      (effects
+        (font (size 1.524 1.524))
+        (justify right)
+      )
+      (uuid "pin-pwr-tps-int-1")
+    )
+    (pin "VBAT+" bidirectional
+      (at 25.4 114.3 180)
+      (effects
+        (font (size 1.524 1.524))
+        (justify left)
+      )
+      (uuid "pin-pwr-vbat-1")
+    )
+  )
   (sheet
     (at 101.6 88.9)
@@
       (uuid "pin-mcu-3v3-1")
     )
-    (pin "I2C_SCL" bidirectional
+    (pin "I2C1_SCL" bidirectional
       (at 152.4 93.98 0)
       (effects
@@
         (justify right)
       )
-      (uuid "pin-i2c-scl-1")
-    )
-    (pin "I2C_SDA" bidirectional
+      (uuid "pin-i2c1-scl-1")
+    )
+    (pin "I2C1_SDA" bidirectional
       (at 152.4 99.06 0)
       (effects
@@
         (justify right)
       )
-      (uuid "pin-i2c-sda-1")
+      (uuid "pin-i2c1-sda-1")
+    )
+    (pin "TPS_INT" input
+      (at 101.6 99.06 180)
+      (effects
+        (font (size 1.524 1.524))
+        (justify left)
+      )
+      (uuid "pin-tps-int-1")
     )
     (pin "PWM_PA" output
@@
     )
   )
-  ;; Sheet: Clock Generator
   (sheet
     (at 177.8 88.9)
@@
       (uuid "pin-clk2-1")
     )
-  )
-  ;; Sheet: RF Section
+    (pin "+3V3" input
+      (at 177.8 104.14 180)
+      (effects
+        (font (size 1.524 1.524))
+        (justify left)
+      )
+      (uuid "pin-clk-3v3-1")
+    )
+    (pin "+5V" input
+      (at 177.8 109.22 180)
+      (effects
+        (font (size 1.524 1.524))
+        (justify left)
+      )
+      (uuid "pin-clk-5v-1")
+    )
+  )
   (sheet
     (at 25.4 139.7)
@@
       (uuid "pin-rf-rxq-1")
     )
-  )
-  ;; Sheet: Debug Interface
+    (pin "TX_EN" input
+      (at 25.4 170.18 180)
+      (effects
+        (font (size 1.524 1.524))
+        (justify left)
+      )
+      (uuid "pin-rf-txen-1")
+    )
+  )
   (sheet
     (at 114.3 139.7)
@@
       (uuid "pin-jtag-tdo-1")
     )
-  )
-  ;; Sheet: USB Connectors
+    (pin "USB2_DP" bidirectional
+      (at 114.3 149.86 180)
+      (effects
+        (font (size 1.524 1.524))
+        (justify left)
+      )
+      (uuid "pin-dbg-usb2-dp-1")
+    )
+    (pin "USB2_DM" bidirectional
+      (at 114.3 154.94 180)
+      (effects
+        (font (size 1.524 1.524))
+        (justify left)
+      )
+      (uuid "pin-dbg-usb2-dm-1")
+    )
+  )
   (sheet
     (at 177.8 139.7)
@@
       )
     )
-    (pin "VBUS_OUT" output
+    (pin "VBUS" output
       (at 215.9 144.78 0)
       (effects
@@
         (justify right)
       )
-      (uuid "pin-usb-vbus-out-1")
+      (uuid "pin-usb-vbus-1")
     )
     (pin "CC1" bidirectional
@@
     )
   )
-  ;; Notes
   (text "JLCPCB Part Selection Notes:\n\n• Basic parts used where possible (0402/0603 R/C)\n• STM32G474RET6 - Extended part (C481410)\n• Si5351A-B-GT - Extended part\n• AMS1117-3.3 - Basic part (C6186)\n• Common MOSFETs: 2N7002 (C8545), SI2302 (C10487)\n• ESD protection: USBLC6-2SC6 (C7519)\n• Crystals: 8MHz HC-49S (C32160), 25MHz (C255909)"
     (exclude_from_sim no)

Commit message: Add Python KiCad helper library and JLCPCB component libraries
- Add kicad_lib: Python library for parsing, creating, and validating KiCad files
  - S-expression parser and writer for .kicad_sym and .kicad_sch files
  - Immutable dataclasses for symbols, schematics, pins, wires, etc.
  - SymbolBuilder with fluent API for programmatic symbol creation
  - ERC validation runner with configurable rules
  - Result type for explicit error handling

- Add custom_lib: JLCPCB component libraries downloaded via JLC2KiCadLib
  - 21 symbol definitions (.kicad_sym)
  - 19 footprints with 3D STEP models
  - Includes STM32G474, TPS25750D, BQ25798, Si5351A, FT4232HL, etc.

- Update CLAUDE.md with kicad_lib documentation and usage examples

- Update schematic sheets with embedded lib_symbols and wiring
Connections:
- no-connect marks 0 -> 12
Other:
- sheet Power_Management ports: added TPS_I2CM_SCL, TPS_I2CM_SDA; removed none

Commit message: schematic is still quite borked
Connections:
- no-connect marks 12 -> 8
Other:
- sheet Clock_Si5351 ports: added none; removed +3V3, +5V
- sheet MCU_STM32G4 ports: added TX_EN; removed TPS_INT
- sheet Power_Management ports: added none; removed TPS_I2CM_SCL, TPS_I2CM_SDA, TPS_INT, VBAT+
- note added: "JLCPCB Part Selection Notes: - Basic parts used where possible (0402/0603 R/C) - STM32G474RET6 - Extended part (C481410) - Si5351A-B-GT - Extended part - AMS1117-3.3 - Basic part (C6186) - Common MOSFETs: 2N7002 (C8545), SI2302 (C10487) - ESD protection: USBLC6-2SC6 (C7519) - Crystals: 8MHz HC-49S (C32160), 25MHz (C255909)"
- note added: "Power Rails: - VBUS: 5-20V (USB-C PD) - VSYS: 9-14V (Battery/Charger) - +5V: Logic, FT4232, Si5351 VDDO - +3V3: MCU, Si5351 core"
- note removed: "JLCPCB Part Selection Notes: • Basic parts used where possible (0402/0603 R/C) • STM32G474RET6 - Extended part (C481410) • Si5351A-B-GT - Extended part • AMS1117-3.3 - Basic part (C6186) • Common MOSFETs: 2N7002 (C8545), SI2302 (C10487) • ESD protection: USBLC6-2SC6 (C7519) • Crystals: 8MHz HC-49S (C32160), 25MHz (C255909)"
- note removed: "Power Rails: • VBUS: 5-20V (USB-C PD) • VSYS: 9-14V (Battery/Charger) • +5V: Logic, FT4232, Si5351 VDDO • +3V3: MCU, Si5351 core"
