File: sdr_kicad/debug_ft4232.kicad_sch (KiCad schematic)
At the start: 9 parts

Commit message: Add Python KiCad helper library and JLCPCB component libraries
- Add kicad_lib: Python library for parsing, creating, and validating KiCad files
  - S-expression parser and writer for .kicad_sym and .kicad_sch files
  - Immutable dataclasses for symbols, schematics, pins, wires, etc.
  - SymbolBuilder with fluent API for programmatic symbol creation
  - ERC validation runner with configurable rules
  - Result type for explicit error handling

- Add custom_lib: JLCPCB component libraries downloaded via JLC2KiCadLib
  - 21 symbol definitions (.kicad_sym)
  - 19 footprints with 3D STEP models
  - Includes STM32G474, TPS25750D, BQ25798, Si5351A, FT4232HL, etc.

- Update CLAUDE.md with kicad_lib documentation and usage examples

- Update schematic sheets with embedded lib_symbols and wiring
Parts:
- added U6: FT4232HL, Package_QFP:LQFP-64_10x10mm_P0.5mm, symbol FT4232HL:FT4232HL-Reel
Changed lines of the file:
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@@
     (uuid "hlabel-usb2-dm")
   )
+  (symbol
+    (lib_id "FT4232HL:FT4232HL-Reel")
+    (at 76.2 76.2 0)
+    (unit 1)
+    (exclude_from_sim no)
+    (in_bom yes)
+    (on_board yes)
+    (dnp no)
+    (uuid "u6-ft4232h")
+    (property "Reference" "U6"
+      (at 76.2 25.4 0)
+      (effects (font (size 1.27 1.27)))
+    )
+    (property "Value" "FT4232HL"
+      (at 76.2 27.94 0)
+      (effects (font (size 1.27 1.27)))
+    )
+    (property "Footprint" "Package_QFP:LQFP-64_10x10mm_P0.5mm"
+      (at 76.2 76.2 0)
+      (effects (font (size 1.27 1.27)) hide)
+    )
+    (property "LCSC" "C2688064"
+      (at 76.2 76.2 0)
+      (effects (font (size 1.27 1.27)) hide)
+    )
+  )
+  (wire
+    (pts (xy 20.32 50.8) (xy 50.8 50.8))
+    (uuid "wire-dbg-5v-1")
+  )
+  (wire
+    (pts (xy 50.8 50.8) (xy 50.8 35.56))
+    (uuid "wire-dbg-5v-2")
+  )
+  (wire
+    (pts (xy 119.38 182.88) (xy 139.7 182.88))
+    (uuid "wire-dbg-tck")
+  )
+  (wire
+    (pts (xy 119.38 193.04) (xy 139.7 193.04))
+    (uuid "wire-dbg-tms")
+  )
+  (wire
+    (pts (xy 119.38 203.2) (xy 139.7 203.2))
+    (uuid "wire-dbg-tdi")
+  )
+  (wire
+    (pts (xy 119.38 213.36) (xy 139.7 213.36))
+    (uuid "wire-dbg-tdo")
+  )
+  (wire
+    (pts (xy 220.98 68.58) (xy 236.22 68.58))
+    (uuid "wire-dbg-usb2dp")
+  )
+  (wire
+    (pts (xy 220.98 81.28) (xy 236.22 81.28))
+    (uuid "wire-dbg-usb2dm")
+  )
 )

Commit message: schematic is still quite borked
Parts:
- FB1: symbol Device:Ferrite_Bead -> Ferrite_Bead:SDFL2012S100KTF
Changed lines of the file:
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@@
   )
   (symbol
-    (lib_id "Device:Ferrite_Bead")
+    (lib_id "Ferrite_Bead:SDFL2012S100KTF")
     (at 190.5 50.8 90)
     (unit 1)

Commit message: add firmware and readme
Parts:
- added unit 3 of U6
- added unit 2 of U6
- added unit 4 of U6
- added unit 5 of U6
Connections:
- net +5V: now also U6.8 (USBDP)
- net JTAG_TDO: now also U6.33 (ADBUS5)
- net GND: now reaches C70.1
- net GND: now also C71.1, U6.20 (VCCIO), U6.31 (VCCIO), U6.37 (VCORE), U6.4 (VPHY), U6.9 (VPLL)
- net +3V3: now reaches C70.2
- net +3V3: now also C71.2, U6.10 (AGND), U6.11 (GND), U6.15 (GND), U6.47 (GND), U6.5 (GND), U6.51 (GND)
- no-connect marks 0 -> 39
