File: sdr_kicad/mcu_stm32g4.kicad_sch (KiCad schematic)
At the start: 10 parts, among them SW1 RESET, Y1 8MHz

Commit message: Add missing schematic symbols and fix hierarchical connections
- Add USB-C receptacles (J1, J2) and USBLC6-2SC6 ESD ICs to usb_connectors
- Add FST3253 QSD, EC2-3SNU relays (K1-K5), SMA connector, 1N5711 diodes to rf_section
- Add missing sheet pins for proper hierarchical signal routing
- Remove invalid comment lines that broke KiCad parser
- Update power management to TPS25750D/BQ25798 architecture for 4S battery support
- ERC reduced from 89 to 82 violations (remaining are unwired connections)
Other:
- note added: "STM32 I2C1 @ 400kHz (Host Bus): • 0x60 - Si5351A (Clock Gen) • 0x21 - TPS25750D (USB-PD, I2CS port) • 0x6B - BQ25798 (Charger, monitoring) • 0x08 - BQ76920 (Battery AFE) • 0x3C - SSD1306 (OLED, optional) TPS25750D I2CM (Charger Control): • 0x6B - BQ25798 (autonomous config) Note: TPS25750D autonomously controls BQ25798 via its I2CM port. STM32 can monitor charger status via shared bus. Pull-ups: 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"
- note added: "STM32G474RET6 Features: • 512KB Flash, 128KB RAM • 170MHz Cortex-M4F with FPU/DSP • USB Full-Speed (UCPD unused) • 5x 12-bit ADC (4 MSPS) • 2x 12-bit DAC • HRTIM for precise PWM • 4x I2C, 4x SPI, 5x UART LCSC Part: C481410 Package: LQFP-64 Pin Assignments (Key): • PA0: PTT Input • PA4: Audio DAC Out • PA11/PA12: USB D-/D+ • PB4: TPS25750D INT (optional) • PB5: GPIO Spare • PB6/PB7: I2C1 SCL/SDA •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"
- note added: "USB Connections: • PA11: USB_DM • PA12: USB_DP Freed UCPD Pins (UCPD not used): • PB4: TPS25750D_INT (optional) • PB5: GPIO_SPARE (reserved) Note: USB Power Delivery is handled by the standalone TPS25750D controller. STM32 UCPD peripheral unused. ESD Protection: USBLC6-2SC6 (C7519) Basic part, protects D+/D-"
- note added: "USB Full-Speed (Data Only)"
- note removed: "I2C1 @ 400kHz: • 0x60 - Si5351A (Clock Gen) • 0x6B - BQ25713 (Charger) • 0x08 - BQ76920 (Battery AFE) • 0x35 - TCPP03-M20 (USB-C) • 0x3C - SSD1306 (OLED, optional) Pull-ups: 2.2k on SCL/SDA LCSC: C25879 (Basic 0402)"
- note removed: "STM32G474RET6 Features: • 512KB Flash, 128KB RAM • 170MHz Cortex-M4F with FPU/DSP • USB Full-Speed + UCPD • 5x 12-bit ADC (4 MSPS) • 2x 12-bit DAC • HRTIM for precise PWM • 4x I2C, 4x SPI, 5x UART LCSC Part: C481410 Package: LQFP-64 Pin Assignments (Key): • PA0: PTT Input • PA4: Audio DAC Out • PA11/PA12: USB D-/D+ • PB4/PB5: UCPD CC1/CC2 • PB6/PB7: I2C1 SCL/SDA • PC0/PC1: ADC (SWR FWD/REV) • PC2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"
- note removed: "USB Connections: • PA11: USB_DM • PA12: USB_DP UCPD Connections: • PB4: UCPD1_CC1 • PB5: UCPD1_CC2 ESD Protection: USBLC6-2SC6 (C7519) Basic part, protects D+/D-"
- note removed: "USB Full-Speed + UCPD"

Commit message: Add Python KiCad helper library and JLCPCB component libraries
- Add kicad_lib: Python library for parsing, creating, and validating KiCad files
  - S-expression parser and writer for .kicad_sym and .kicad_sch files
  - Immutable dataclasses for symbols, schematics, pins, wires, etc.
  - SymbolBuilder with fluent API for programmatic symbol creation
  - ERC validation runner with configurable rules
  - Result type for explicit error handling

- Add custom_lib: JLCPCB component libraries downloaded via JLC2KiCadLib
  - 21 symbol definitions (.kicad_sym)
  - 19 footprints with 3D STEP models
  - Includes STM32G474, TPS25750D, BQ25798, Si5351A, FT4232HL, etc.

- Update CLAUDE.md with kicad_lib documentation and usage examples

- Update schematic sheets with embedded lib_symbols and wiring
Parts:
- added U1: STM32G474RETx, Package_QFP:LQFP-64_10x10mm_P0.5mm, symbol STM32G474RET6:STM32G474RET6
Other:
- note added: "MCU Pin Connections: • PA12 → USB_DP (via ESD) • PA11 → USB_DM (via ESD) • PC6 → PWM_PA (HRTIM) • PB4 → TPS_INT (GPIO input) • PA1-3, PA6-7, PB8-12 → BAND_SEL bus"
Changed lines of the file:
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@@
     )
+  )
+  (symbol
+    (lib_id "STM32G474RET6:STM32G474RET6")
+    (at 101.6 101.6 0)
+    (unit 1)
+    (exclude_from_sim no)
+    (in_bom yes)
+    (on_board yes)
+    (dnp no)
+    (uuid "u1-stm32g474")
+    (property "Reference" "U1"
+      (at 101.6 38.1 0)
+      (effects (font (size 1.27 1.27)))
+    )
+    (property "Value" "STM32G474RETx"
+      (at 101.6 40.64 0)
+      (effects (font (size 1.27 1.27)))
+    )
+    (property "Footprint" "Package_QFP:LQFP-64_10x10mm_P0.5mm"
+      (at 101.6 101.6 0)
+      (effects (font (size 1.27 1.27)) hide)
+    )
+    (property "LCSC" "C481410"
+      (at 101.6 101.6 0)
+      (effects (font (size 1.27 1.27)) hide)
+    )
+  )
+  (symbol
+    (lib_id "power:+3V3")
+    (at 25.4 45.72 0)
+    (unit 1)
+    (exclude_from_sim no)
+    (in_bom no)
+    (on_board yes)
+    (dnp no)
+    (uuid "pwr-mcu-3v3")
+    (property "Reference" "#PWR06"
+      (at 25.4 49.53 0)
+      (effects (font (size 1.27 1.27)) hide)
+    )
+    (property "Value" "+3V3"
+      (at 25.4 41.91 0)
+      (effects (font (size 1.27 1.27)))
+    )
+  )
+  (wire
+    (pts
+      (xy 25.4 45.72)
+      (xy 25.4 50.8)
+    )
+    (uuid "wire-mcu-3v3")
+  )
+  (wire
+    (pts
+      (xy 368.3 76.2)
+      (xy 381 76.2)
+    )
+    (uuid "wire-mcu-scl")
+  )
+  (wire
+    (pts
+      (xy 368.3 88.9)
+      (xy 381 88.9)
+    )
+    (uuid "wire-mcu-sda")
   )
   (hierarchical_label "+3V3"
@@
     (uuid "hlabel-tps-int")
   )
+  (wire (pts (xy 139.7 99.06) (xy 300 99.06)) (uuid "wire-mcu-pwm-1"))
+  (wire (pts (xy 300 99.06) (xy 300 101.6)) (uuid "wire-mcu-pwm-2"))
+  (wire (pts (xy 300 101.6) (xy 381 101.6)) (uuid "wire-mcu-pwm-3"))
+  (bus (pts (xy 139.7 114.3) (xy 381 114.3)) (uuid "bus-mcu-band"))
+  (wire (pts (xy 139.7 91.44) (xy 320 91.44)) (uuid "wire-mcu-usb-dp-1"))
+  (wire (pts (xy 320 91.44) (xy 320 127)) (uuid "wire-mcu-usb-dp-2"))
+  (wire (pts (xy 320 127) (xy 381 127)) (uuid "wire-mcu-usb-dp-3"))
+  (wire (pts (xy 139.7 93.98) (xy 315 93.98)) (uuid "wire-mcu-usb-dm-1"))
+  (wire (pts (xy 315 93.98) (xy 315 139.7)) (uuid "wire-mcu-usb-dm-2"))
+  (wire (pts (xy 315 139.7) (xy 381 139.7)) (uuid "wire-mcu-usb-dm-3"))
+  (wire (pts (xy 63.5 109.22) (xy 50.8 109.22)) (uuid "wire-mcu-tps-int-1"))
+  (wire (pts (xy 50.8 109.22) (xy 50.8 180)) (uuid "wire-mcu-tps-int-2"))
+  (wire (pts (xy 50.8 180) (xy 350 180)) (uuid "wire-mcu-tps-int-3"))
+  (wire (pts (xy 350 180) (xy 350 152.4)) (uuid "wire-mcu-tps-int-4"))
+  (wire (pts (xy 350 152.4) (xy 381 152.4)) (uuid "wire-mcu-tps-int-5"))
+  (text "MCU Pin Connections:\n• PA12 → USB_DP (via ESD)\n• PA11 → USB_DM (via ESD)\n• PC6  → PWM_PA (HRTIM)\n• PB4  → TPS_INT (GPIO input)\n• PA1-3, PA6-7, PB8-12 → BAND_SEL bus"
+    (exclude_from_sim no)
+    (at 280 180 0)
+    (effects (font (size 1.27 1.27)) (justify left))
+    (uuid "text-mcu-pin-notes")
+  )
 )

Commit message: schematic is still quite borked
Parts:
- removed C12: 100nF, Capacitor_SMD:C_0402_1005Metric, symbol Device:C
- removed C13: 4.7uF, Capacitor_SMD:C_0402_1005Metric, symbol Device:C
- added C20: 4.7uF, Capacitor_SMD:C_0402_1005Metric, symbol Device:C
- added C21: 100nF, Capacitor_SMD:C_0402_1005Metric, symbol Device:C
- added FB1: 600R@100MHz, Inductor_SMD:L_0402_1005Metric, symbol Device:L_Ferrite
- C10, C11, C14, R10, R20, R21, Y1: JLC_Basic Yes -> (none)
- SW1: symbol Switch:SW_Push -> sdr_components:TS-1187A-B-A-B
Connections:
- net +3V3: now also C10.1, C10.2, C11.1, C11.2, C14.1, C14.2, R10.1, R10.2, R20.1, R21.1, U1.1 (VBAT), U1.15 (VSS), U1.16 (VDD), U1.27 (VSSA), U1.28 (VREF+), U1.29 (VDDA), U1.31 (VSS), U1.32 (VDD), U1.47 (VSS), U1.48 (VDD), U1.5 (PF0-OSC_IN), U1.6 (PF1-OSC_OUT), U1.61 (PB8-BOOT0), U1.63 (VSS), U1.64 (VDD), U1.7 (PG10-NRST), Y1.1, Y1.2, C20.1, C20.2, C21.1, C21.2, FB1.1, FB1.2
- net I2C1_SCL: now also R20.2, U1.59 (PB6)
- net I2C1_SDA: now also R21.2, U1.60 (PB7)
- net PWM_PA: now also U1.42 (PA8)
- net USB_DM: now also U1.45 (PA11)
- net USB_DP: now also U1.46 (PA12)
- net SWDIO: now reaches U1.49 (PA13)
- net SWCLK: now reaches U1.50 (PA14)
- no-connect marks 0 -> 41
Other:
- note removed: "8MHz HSE Crystal"
- note removed: "ADC Channels: • PC0 (ADC1_IN6): SWR Forward • PC1 (ADC1_IN7): SWR Reverse • PC2 (ADC1_IN8): Audio Input • PB0 (ADC1_IN15): Battery Voltage DAC Channels: • PA4 (DAC1_OUT1): Audio Output • PA5 (DAC1_OUT2): Spare/Reference Op-Amp (for Audio): LM358 or similar LCSC: C7950 (Basic)"
- note removed: "Analog Inputs"
- note removed: "GPIO Pin Assignments"
- note removed: "I2C1 Bus Devices"
- note removed: "MCU Pin Connections: • PA12 → USB_DP (via ESD) • PA11 → USB_DM (via ESD) • PC6 → PWM_PA (HRTIM) • PB4 → TPS_INT (GPIO input) • PA1-3, PA6-7, PB8-12 → BAND_SEL bus"
- note removed: "Port A: PA0 - PTT Input (EXTI) PA1 - Band Relay SET 0 PA2 - Band Relay SET 1 PA3 - Band Relay SET 2 PA4 - DAC1_OUT1 (Audio Out) PA5 - DAC1_OUT2 PA6 - Band Relay RESET 0 PA7 - Band Relay RESET 1 PA8 - MCO1 (Debug Clock Out) PA9 - USART1_TX PA10 - USART1_RX PA11 - USB_DM PA12 - USB_DP PA13 - SWDIO PA14 - SWCLK PA15 - JTAG_TDI Port B: PB0 - ADC (VBAT Sense) PB1 - TX Enable PB2 - BOOT0 (tie low) PB3 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"
- note removed: "Power Decoupling"
- note removed: "Reset Circuit"
- note removed: "STM32 I2C1 @ 400kHz (Host Bus): • 0x60 - Si5351A (Clock Gen) • 0x21 - TPS25750D (USB-PD, I2CS port) • 0x6B - BQ25798 (Charger, monitoring) • 0x08 - BQ76920 (Battery AFE) • 0x3C - SSD1306 (OLED, optional) TPS25750D I2CM (Charger Control): • 0x6B - BQ25798 (autonomous config) Note: TPS25750D autonomously controls BQ25798 via its I2CM port. STM32 can monitor charger status via shared bus. Pull-ups: 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"
- note removed: "STM32G474RET6 Features: • 512KB Flash, 128KB RAM • 170MHz Cortex-M4F with FPU/DSP • USB Full-Speed (UCPD unused) • 5x 12-bit ADC (4 MSPS) • 2x 12-bit DAC • HRTIM for precise PWM • 4x I2C, 4x SPI, 5x UART LCSC Part: C481410 Package: LQFP-64 Pin Assignments (Key): • PA0: PTT Input • PA4: Audio DAC Out • PA11/PA12: USB D-/D+ • PB4: TPS25750D INT (optional) • PB5: GPIO Spare • PB6/PB7: I2C1 SCL/SDA •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"
- note removed: "USB Connections: • PA11: USB_DM • PA12: USB_DP Freed UCPD Pins (UCPD not used): • PB4: TPS25750D_INT (optional) • PB5: GPIO_SPARE (reserved) Note: USB Power Delivery is handled by the standalone TPS25750D controller. STM32 UCPD peripheral unused. ESD Protection: USBLC6-2SC6 (C7519) Basic part, protects D+/D-"
- note removed: "USB Full-Speed (Data Only)"
- note removed: "VDD Decoupling (x4): 100nF 0402 on each VDD pin LCSC: C1525 (Basic) VDDA Decoupling: 4.7uF + 100nF LCSC: C23733 + C1525 VCAP: 2x 1uF on VCAP1/VCAP2 LCSC: C52923"
- moved on the sheet: C10, C11, C14, R10, R20, R21, Y1

Commit message: add firmware and readme
Connections:
- net SWCLK is gone; now on net +3V3: U1.50 (PA14)
- net SWDIO is gone; now on net +3V3: U1.49 (PA13)
- net +3V3: now also U1.17 (PA3), U1.18 (PA4), U1.19 (PA5), U1.2 (PC13), U1.20 (PA6), U1.21 (PA7), U1.22 (PC4), U1.23 (PC5), U1.24 (PB0), U1.25 (PB1), U1.26 (PB2), U1.30 (PB10), U1.33 (PB11), U1.34 (PB12), U1.37 (PB15), U1.38 (PC6), U1.4 (PC15-OSC32_OUT), U1.9 (PC1)
- net PWM_PA: no longer U1.42 (PA8)
- net ENCODER_PUSH: now reaches U1.10 (PC2)
- net ENCODER_B: now reaches U1.11 (PC3)
- net BAND_RESET_1: now reaches U1.12 (PA0)
- net BAND_RESET_0: now reaches U1.13 (PA1)
- net DAC_SPARE: now reaches U1.14 (PA2)
- net BAND_RESET_3: now reaches U1.3 (PC14-OSC32_IN)
- net BAND_SET_3: now reaches U1.35 (PB13)
- net BAND_RESET_2: now reaches U1.36 (PB14)
- net GPIO_SPARE: now reaches U1.39 (PC7)
- net JTAG_TDO_SWO: now reaches U1.41 (PC9)
- net SPI3_MOSI_FLASH: now reaches U1.43 (PA9)
- net UART4_RX_CAT: now reaches U1.44 (PA10)
- net USART1_RX: now reaches U1.53 (PC11)
- net USART1_TX: now reaches U1.54 (PC12)
- net MCO1_DEBUG: now reaches U1.55 (PD2)
- net LED_STATUS: now reaches U1.56 (PB3)
- net TR_SWITCH: now reaches U1.57 (PB4)
- net HRTIM1_CH2: now reaches U1.58 (PB5)
- net SPI2_SCK: now reaches U1.62 (PB9)
- net TX_ENABLE: now reaches U1.8 (PC0)
- net I2C1_SCL renamed HRTIM1_CH1_PWM_PA
- net USB_DM renamed UART4_TX_CAT
- net USB_DP renamed JTAG_TDI
- new net SPI3_MISO_FLASH: U1.42 (PA8)
Other:
- note added: "MCU Pin Connections: • PA12 → USB_DP (via ESD) • PA11 → USB_DM (via ESD) • PC6 → PWM_PA (HRTIM) • PB4 → TPS_INT (GPIO input) • PA1-3, PA6-7, PB8-12 → BAND_SEL bus"
