File: sdr_kicad/power_management.kicad_sch (KiCad schematic)
At the start: 11 parts

Commit message: Add missing schematic symbols and fix hierarchical connections
- Add USB-C receptacles (J1, J2) and USBLC6-2SC6 ESD ICs to usb_connectors
- Add FST3253 QSD, EC2-3SNU relays (K1-K5), SMA connector, 1N5711 diodes to rf_section
- Add missing sheet pins for proper hierarchical signal routing
- Remove invalid comment lines that broke KiCad parser
- Update power management to TPS25750D/BQ25798 architecture for 4S battery support
- ERC reduced from 89 to 82 violations (remaining are unwired connections)
Parts:
- removed R1, R2: 5.1k, Resistor_SMD:R_0402_1005Metric, symbol Device:R
- added C3: 2.2uF/10V, Capacitor_SMD:C_0402_1005Metric, symbol Device:C
- added C4: 100nF, Capacitor_SMD:C_0402_1005Metric, symbol Device:C
- added C5, C6, C7, C8, C9: 22uF/25V, Capacitor_SMD:C_0805_2012Metric, symbol Device:C
- added L2: 68uH, Inductor_SMD:L_6.3x6.3_H3, symbol Device:L
- L1: value 2.2uH/5A -> 1.5uH/10A; LCSC C408412 -> C2827517
- renumbered C5 to C10, C6 to C11, C7 to C12, R3 to R1
Other:
- note added: "5V Buck Regulator (XL1509-5.0E1)"
- note added: "AMS1117-3.3 (JLCPCB Basic) LCSC: C6186 • Fixed 3.3V Output • 1A Output Current • SOT-223 Package IMPORTANT: Input from +5V rail (NOT from VSYS - 4S voltage too high) Dropout: 5V - 3.3V = 1.7V headroom Capacitors: • Cin: 10uF ceramic (C11) • Cout: 22uF ceramic (C12)"
- note added: "BQ25798 Configuration: • 1-4S Li-Ion/LiPo Charger • Buck-Boost Topology (NVDC) • Integrated Power FETs (no external MOSFETs) • Integrated BATFET • I2C Interface (Addr: 0x6B) • Autonomous charging mode • Input: 3.6V - 24V • Charge Current: Up to 5A • Supports USB PD 3.0 PPS LCSC Part: C2876593 Key External Components: • Input Cap: 2x 22uF/25V (C5, C6) • Output Cap: 2x 22uF/25V (C7, C8) • Inductor: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"
- note added: "BQ76920 Features: • 3-5 Series Cell Support (using 4S) • Integrated Cell Balancing • Coulomb Counter • I2C Interface (Addr: 0x08) • OVP/UVP/OCP/SCP Protection LCSC Part: C82092 4S Protection Thresholds: • OV: 4.25V/cell (17.0V pack max) • UV: 2.8V/cell (11.2V pack min) • OCD: 10A • SCD: 50A • OCP Charge: 5A 4S Pack Voltage Range: • Nominal: 14.8V (3.7V/cell) • Full: 16.8V (4.2V/cell) • Empty: 12.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"
- note added: "Battery Monitor AFE (BQ76920) - 4S Configuration"
- note added: "Buck-Boost Battery Charger (BQ25798RQMR)"
- note added: "I2C BUS ARCHITECTURE TPS25750D I2CM (Charger Control - Autonomous): └─► BQ25798 (0x6B) - Charger configuration STM32 I2C1 @ 400kHz (Host Bus): ├─► Si5351A (0x60) - Clock synthesizer ├─► TPS25750D I2CS (0x21) - PD monitoring ├─► BQ25798 (0x6B) - Charger status read ├─► BQ76920 (0x08) - Battery AFE └─► SSD1306 (0x3C) - OLED display (optional) Note: TPS25750D autonomously configures BQ25798 via its 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"
- note added: "JLCPCB PART NUMBERS (Basic = B, Extended = E) Power Management ICs (Extended): • TPS25750DRJKR: C2868209 (USB-PD Controller) • BQ25798RQMR: C2876593 (Buck-Boost Charger) • BQ76920PW: C82092 (Battery AFE) Regulators (Basic): • XL1509-5.0E1: C61063 (5V Buck) • AMS1117-3.3: C6186 (3.3V LDO) Passives (Basic): • 0402 100nF: C1525 • 0603 10uF: C19702 • 0805 22uF/25V: C45783 • 0402 2.2uF: C52923 • SS34 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"
- note added: "POWER DISTRIBUTION SUMMARY (4S Architecture) VBUS (USB-C): 5-20V from PD negotiation └─► TPS25750D VBUS input └─► PP_HV (power path) ──► BQ25798 VAC1 VSYS (12-18V): Output from BQ25798 SYS pin ├─► H-Bridge PA (uP9636) [VERIFY: VCC max >= 18V] └─► 5V Buck Input (XL1509, rated 4.5-40V) ──► OK VBAT (12.8-16.8V): 4S Li-Ion Pack ├─► BQ76920 Cell Monitoring (3-5S capable) └─► BQ25798 BAT Port +5V (5.0V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"
- note added: "TPS25750D Features: • Standalone USB Type-C and PD Controller • No MCU firmware required for PD negotiation • Integrated 28V/7A power path switch • Integrated CC protection (no TCPP03 needed) • I2C Master port for autonomous charger control • I2C Slave port for host monitoring • Dead battery boot support • Web GUI configuration tool LCSC Part: C2868209 I2C Slave Address: 0x21 Configuration: • Sin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"
- note added: "TPS25750D Signal Flow: USB-C Connector: CC1/CC2 --> TPS25750D (direct, internal Rd) VBUS --> TPS25750D VBUS pin TPS25750D Outputs: PP_HV (28V/7A switch) --> BQ25798 VAC1 I2CM_SCL/SDA --> BQ25798 I2C (charger control) I2CS_SCL/SDA --> STM32 I2C1 (host monitoring) INT# --> STM32 GPIO (optional alert)"
- note added: "USB-C PD Controller (TPS25750DRJKR)"
- note added: "XL1509-5.0E1 (JLCPCB Basic) LCSC: C61063 • Fixed 5V Output • 2A Output Current • Input: 4.5V-40V (OK for 4S 18V max) Components: • Cin: 22uF/25V (C9) • Cout: 22uF/10V (C10) • L: 68uH (L2) • D: SS34 Schottky (D1)"
- note removed: "5V Buck Regulator (TPS62160 or XL1509)"
- note removed: "AMS1117-3.3 (JLCPCB Basic) LCSC: C6186 • Fixed 3.3V Output • 1A Output Current • Input: 4.5V-15V • SOT-223 Package Capacitors: • Cin: 10uF ceramic • Cout: 22uF ceramic"
- note removed: "Alternative JLCPCB Basic: XL1509-5.0E1 (C61063) • Fixed 5V Output • 2A Output Current • Input: 4.5V-40V Components: • Cin: 22uF/25V • Cout: 22uF/10V • L: 68uH • D: SS34 Schottky"
- note removed: "BQ25713 Configuration: • 1-4S Li-Ion/LiPo Charger • Buck-Boost Topology (NVDC) • I2C Interface (Addr: 0x6B) • USB PD 3.0 Compatible • Input: 3.5V - 24V • Charge Current: Up to 8A Key External Components: • Input Cap: 22uF/25V (C1) • Output Cap: 22uF/25V (C2) • Inductor: 2.2uH/5A (L1) • Sense Resistor: 10mOhm (R_SNS)"
- note removed: "BQ76920 Features: • 3-5 Series Cell Support • Integrated Cell Balancing • Coulomb Counter • I2C Interface (Addr: 0x08) • OVP/UVP/OCP/SCP Protection LCSC Part: C82092 Protection Thresholds: • OV: 4.25V/cell • UV: 2.8V/cell • OCD: 10A • SCD: 50A"
- note removed: "Battery Monitor AFE (BQ76920)"
- note removed: "Buck-Boost Battery Charger (BQ25713RSNR)"
- note removed: "JLCPCB PART NUMBERS (Basic = B, Extended = E) Passives: • 0402 10k: C25744 (B) • 0402 5.1k: C25905 (B) • 0402 100nF: C1525 (B) • 0603 10uF: C19702 (B) • 0805 22uF: C45783 (B) • 0402 4.7uF: C23733 (B) Semiconductors: • AMS1117-3.3: C6186 (B) • SS34 Schottky: C8678 (B) • 2N7002: C8545 (B) • SI2302: C10487 (B) ICs (Extended): • STM32G474RET6: C481410 • BQ25713RSNR: C134263 • BQ76920PW: C82092 • Si53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"
- note removed: "Note: TCPP03-M20 (LCSC: C2682766) Provides CC protection, VBUS control, and dead battery support. Connects to STM32G4 UCPD pins."
- note removed: "POWER DISTRIBUTION SUMMARY VBUS (USB-C): 5-20V from PD negotiation └─► BQ25713 Input VSYS (9-14V): Output from BQ25713 NVDC ├─► H-Bridge PA (uP9636) ├─► 5V Buck Input └─► 3.3V LDO Input (if VSYS < 15V) VBAT (9.6-12.6V): 3S Li-Ion Pack ├─► BQ76920 Cell Monitoring └─► BQ25713 Battery Port +5V (5.0V): From Buck Regulator ├─► FT4232H ├─► Si5351A VDDO └─► Relay Driver Supply +3V3 (3.3V): From AMS1117-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"
- note removed: "USB-C Port Protection (TCPP03-M20)"

Commit message: Add Python KiCad helper library and JLCPCB component libraries
- Add kicad_lib: Python library for parsing, creating, and validating KiCad files
  - S-expression parser and writer for .kicad_sym and .kicad_sch files
  - Immutable dataclasses for symbols, schematics, pins, wires, etc.
  - SymbolBuilder with fluent API for programmatic symbol creation
  - ERC validation runner with configurable rules
  - Result type for explicit error handling

- Add custom_lib: JLCPCB component libraries downloaded via JLC2KiCadLib
  - 21 symbol definitions (.kicad_sym)
  - 19 footprints with 3D STEP models
  - Includes STM32G474, TPS25750D, BQ25798, Si5351A, FT4232HL, etc.

- Update CLAUDE.md with kicad_lib documentation and usage examples

- Update schematic sheets with embedded lib_symbols and wiring
Parts:
- removed C1, C2, C5, C6, C7, C8, C9: 22uF/25V, Capacitor_SMD:C_0805_2012Metric, symbol Device:C
- removed C10: 22uF/10V, Capacitor_SMD:C_0805_2012Metric, symbol Device:C
- removed C11: 10uF, Capacitor_SMD:C_0603_1608Metric, symbol Device:C
- removed C12: 22uF, Capacitor_SMD:C_0805_2012Metric, symbol Device:C
- removed C3: 2.2uF/10V, Capacitor_SMD:C_0402_1005Metric, symbol Device:C
- removed C4: 100nF, Capacitor_SMD:C_0402_1005Metric, symbol Device:C
- removed D1: SS34, Diode_SMD:D_SMA, symbol Device:D_Schottky
- removed L1: 1.5uH/10A, Inductor_SMD:L_Bourns_SRN6045, symbol Device:L
- removed L2: 68uH, Inductor_SMD:L_6.3x6.3_H3, symbol Device:L
- removed R1: 10mR/1W, Resistor_SMD:R_2512_6332Metric, symbol Device:R
- removed TH1: 10k NTC, Resistor_SMD:R_0402_1005Metric, symbol Device:Thermistor_NTC
- added U3: AMS1117-3.3, Package_TO_SOT_SMD:SOT-223-3_TabPin2, symbol AMS1117:AMS1117-3_3
- added U4: TPS25750DRJKR, footprint:QFN-38_L6.0-W4.0-P0.40-TL-EP_RJK, symbol TPS25750DRJKR:TPS25750DRJKR
- added U5: BQ25798RQMR, footprint:QFN-29_L4.0-W4.0-P0.40-TL-BQ25792RQMR, symbol BQ25798RQMR:BQ25798RQMR
- added U7: XL1509-5.0E1, footprint:SOIC-8_L5.0-W4.0-P1.27-LS6.0-BL, symbol XL1509:XL1509-5_0E1
Connections:
- net CC1: now also U4.33 (VBUS)
- net CC2: now also U4.32 (VBUS)
- net I2C1_SDA: now also U4.13 (GPIO11)
- net TPS_I2CM_SCL: now also U4.4 (LDO_1V5)
- net TPS_I2CM_SDA: now also U4.5 (GPIO0)
- net TPS_INT: now also U4.11 (GND)
- net VBAT+: now also U5.20 (PROG)
- net VBUS: now also U4.38 (VIN_3V3)
- net VSYS: now also U5.17 (ILIM_HIZ)
- new net GND: U7.5 (GND), U7.8 (GND)
Other:
- note removed: "AMS1117-3.3 (JLCPCB Basic) LCSC: C6186 • Fixed 3.3V Output • 1A Output Current • SOT-223 Package IMPORTANT: Input from +5V rail (NOT from VSYS - 4S voltage too high) Dropout: 5V - 3.3V = 1.7V headroom Capacitors: • Cin: 10uF ceramic (C11) • Cout: 22uF ceramic (C12)"
- note removed: "BQ25798 Configuration: • 1-4S Li-Ion/LiPo Charger • Buck-Boost Topology (NVDC) • Integrated Power FETs (no external MOSFETs) • Integrated BATFET • I2C Interface (Addr: 0x6B) • Autonomous charging mode • Input: 3.6V - 24V • Charge Current: Up to 5A • Supports USB PD 3.0 PPS LCSC Part: C2876593 Key External Components: • Input Cap: 2x 22uF/25V (C5, C6) • Output Cap: 2x 22uF/25V (C7, C8) • Inductor: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"
- note removed: "BQ76920 Features: • 3-5 Series Cell Support (using 4S) • Integrated Cell Balancing • Coulomb Counter • I2C Interface (Addr: 0x08) • OVP/UVP/OCP/SCP Protection LCSC Part: C82092 4S Protection Thresholds: • OV: 4.25V/cell (17.0V pack max) • UV: 2.8V/cell (11.2V pack min) • OCD: 10A • SCD: 50A • OCP Charge: 5A 4S Pack Voltage Range: • Nominal: 14.8V (3.7V/cell) • Full: 16.8V (4.2V/cell) • Empty: 12.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"
- note removed: "Battery Monitor AFE (BQ76920) - 4S Configuration"
- note removed: "I2C BUS ARCHITECTURE TPS25750D I2CM (Charger Control - Autonomous): └─► BQ25798 (0x6B) - Charger configuration STM32 I2C1 @ 400kHz (Host Bus): ├─► Si5351A (0x60) - Clock synthesizer ├─► TPS25750D I2CS (0x21) - PD monitoring ├─► BQ25798 (0x6B) - Charger status read ├─► BQ76920 (0x08) - Battery AFE └─► SSD1306 (0x3C) - OLED display (optional) Note: TPS25750D autonomously configures BQ25798 via its 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"
- note removed: "JLCPCB PART NUMBERS (Basic = B, Extended = E) Power Management ICs (Extended): • TPS25750DRJKR: C2868209 (USB-PD Controller) • BQ25798RQMR: C2876593 (Buck-Boost Charger) • BQ76920PW: C82092 (Battery AFE) Regulators (Basic): • XL1509-5.0E1: C61063 (5V Buck) • AMS1117-3.3: C6186 (3.3V LDO) Passives (Basic): • 0402 100nF: C1525 • 0603 10uF: C19702 • 0805 22uF/25V: C45783 • 0402 2.2uF: C52923 • SS34 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"
- note removed: "POWER DISTRIBUTION SUMMARY (4S Architecture) VBUS (USB-C): 5-20V from PD negotiation └─► TPS25750D VBUS input └─► PP_HV (power path) ──► BQ25798 VAC1 VSYS (12-18V): Output from BQ25798 SYS pin ├─► H-Bridge PA (uP9636) [VERIFY: VCC max >= 18V] └─► 5V Buck Input (XL1509, rated 4.5-40V) ──► OK VBAT (12.8-16.8V): 4S Li-Ion Pack ├─► BQ76920 Cell Monitoring (3-5S capable) └─► BQ25798 BAT Port +5V (5.0V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"
- note removed: "TPS25750D Features: • Standalone USB Type-C and PD Controller • No MCU firmware required for PD negotiation • Integrated 28V/7A power path switch • Integrated CC protection (no TCPP03 needed) • I2C Master port for autonomous charger control • I2C Slave port for host monitoring • Dead battery boot support • Web GUI configuration tool LCSC Part: C2868209 I2C Slave Address: 0x21 Configuration: • Sin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"
- note removed: "TPS25750D Signal Flow: USB-C Connector: CC1/CC2 --> TPS25750D (direct, internal Rd) VBUS --> TPS25750D VBUS pin TPS25750D Outputs: PP_HV (28V/7A switch) --> BQ25798 VAC1 I2CM_SCL/SDA --> BQ25798 I2C (charger control) I2CS_SCL/SDA --> STM32 I2C1 (host monitoring) INT# --> STM32 GPIO (optional alert)"
- note removed: "XL1509-5.0E1 (JLCPCB Basic) LCSC: C61063 • Fixed 5V Output • 2A Output Current • Input: 4.5V-40V (OK for 4S 18V max) Components: • Cin: 22uF/25V (C9) • Cout: 22uF/10V (C10) • L: 68uH (L2) • D: SS34 Schottky (D1)"

Commit message: schematic is still quite borked
Connections:
- net +3V3: now also U3.2 (VOUT), U3.4 (VOUT), U4.1 (LDO_3V3), U4.38 (VIN_3V3)
- net +5V: now also U3.3 (VIN), U7.1 (VIN), U7.2 (OUTPUT)
- net CC1: now also U4.28 (CC1); no longer U4.33 (VBUS)
- net CC2: now also U4.29 (CC2); no longer U4.32 (VBUS)
- net GND: now also U3.1 (GND), U4.11 (GND), U4.12 (GND), U4.14 (GND), U4.31 (GND), U4.39 (GND), U5.27 (GND), U7.6 (GND), U7.7 (GND)
- net I2C1_SCL: now also U4.9 (I2Cs_SCL)
- net I2C1_SDA: now also U4.8 (I2Cs_SDA); no longer U4.13 (GPIO11)
- net TPS_I2CM_SCL: now also U4.17 (I2Cm_SCL); no longer U4.4 (LDO_1V5)
- net TPS_I2CM_SDA: now also U4.16 (I2Cm_SDA); no longer U4.5 (GPIO0)
- net TPS_INT: now also U4.10 (I2Cs_IRQ); no longer U4.11 (GND)
- net VBAT+: now also U5.22 (BAT), U5.23 (BAT); no longer U5.20 (PROG)
- net VBUS: now also U4.23 (VBUS_IN), U4.24 (VBUS_IN), U4.25 (VBUS_IN), U4.32 (VBUS), U4.33 (VBUS), U5.2 (VBUS), U5.3 (VBUS); no longer U4.38 (VIN_3V3)
- net VSYS: now also U5.25 (SYS); no longer U5.17 (ILIM_HIZ)
- net BQ_SCL: now reaches U5.14 (SCL)
- net BQ_SDA: now reaches U5.15 (SDA)
- net BQ_INT: now reaches U5.21 (INT#)
- no-connect marks 0 -> 43

Commit message: add firmware and readme
Connections:
- net +3V3: no longer U3.2 (VOUT), U3.4 (VOUT)
- no-connect marks 43 -> 0
Changed lines of the file:
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@@
   (wire (pts (xy 224.79 175.26) (xy 229.87 175.26)) (uuid "w-ams-gnd2"))
   (junction (at 224.79 175.26) (uuid "j-ams-gnd"))
-  (wire (pts (xy 252.73 177.8) (xy 259.08 177.8)) (uuid "w-ams-vout4"))
-  (wire (pts (xy 259.08 177.8) (xy 259.08 180.34)) (uuid "w-ams-pwrflag"))
-  (wire (pts (xy 259.08 177.8) (xy 264.16 177.8)) (uuid "w-ams-3v3-hl"))
-  (junction (at 259.08 177.8) (uuid "j-ams-3v3"))
-  (wire (pts (xy 229.87 177.8) (xy 229.87 168.91)) (uuid "w-ams-vout2-up"))
-  (wire (pts (xy 229.87 168.91) (xy 256.54 168.91)) (uuid "w-ams-vout2-across"))
-  (wire (pts (xy 256.54 168.91) (xy 256.54 177.8)) (uuid "w-ams-vout2-down"))
-  (wire (pts (xy 256.54 177.8) (xy 259.08 177.8)) (uuid "w-ams-vout2-join"))
-  (no_connect (at 83.82 54.61) (uuid "nc-tps-adcin1"))
-  (no_connect (at 83.82 57.15) (uuid "nc-tps-adcin2"))
-  (no_connect (at 83.82 59.69) (uuid "nc-tps-ldo1v5"))
-  (no_connect (at 83.82 62.23) (uuid "nc-tps-gpio0"))
-  (no_connect (at 83.82 64.77) (uuid "nc-tps-gpio1"))
-  (no_connect (at 83.82 67.31) (uuid "nc-tps-gpio2"))
-  (no_connect (at 83.82 82.55) (uuid "nc-tps-gpio11"))
-  (no_connect (at 83.82 87.63) (uuid "nc-tps-drain15"))
-  (no_connect (at 83.82 95.25) (uuid "nc-tps-i2cm-irq"))
-  (no_connect (at 83.82 97.79) (uuid "nc-tps-gpio3"))
-  (no_connect (at 83.82 100.33) (uuid "nc-tps-pphv20"))
-  (no_connect (at 119.38 52.07) (uuid "nc-tps-drain40"))
-  (no_connect (at 119.38 59.69) (uuid "nc-tps-gpio6"))
-  (no_connect (at 119.38 62.23) (uuid "nc-tps-gpio7"))
-  (no_connect (at 119.38 64.77) (uuid "nc-tps-pp5v35"))
-  (no_connect (at 119.38 67.31) (uuid "nc-tps-pp5v34"))
-  (no_connect (at 119.38 77.47) (uuid "nc-tps-drain30"))
-  (no_connect (at 119.38 85.09) (uuid "nc-tps-usbn"))
-  (no_connect (at 119.38 87.63) (uuid "nc-tps-usbp"))
-  (no_connect (at 119.38 97.79) (uuid "nc-tps-pphv22"))
-  (no_connect (at 119.38 100.33) (uuid "nc-tps-pphv21"))
-  (no_connect (at 224.79 58.42) (uuid "nc-bq-stat"))
-  (no_connect (at 224.79 66.04) (uuid "nc-bq-btst1"))
-  (no_connect (at 224.79 68.58) (uuid "nc-bq-regn"))
-  (no_connect (at 224.79 71.12) (uuid "nc-bq-dp"))
-  (no_connect (at 224.79 73.66) (uuid "nc-bq-dm"))
-  (no_connect (at 224.79 76.2) (uuid "nc-bq-vac2"))
-  (no_connect (at 224.79 78.74) (uuid "nc-bq-vac1"))
-  (no_connect (at 224.79 81.28) (uuid "nc-bq-acdrv2"))
-  (no_connect (at 224.79 83.82) (uuid "nc-bq-acdrv1"))
-  (no_connect (at 224.79 86.36) (uuid "nc-bq-qon"))
-  (no_connect (at 224.79 88.9) (uuid "nc-bq-ce"))
-  (no_connect (at 257.81 55.88) (uuid "nc-bq-pmid"))
-  (no_connect (at 257.81 58.42) (uuid "nc-bq-sw1"))
-  (no_connect (at 257.81 63.5) (uuid "nc-bq-sw2"))
-  (no_connect (at 257.81 68.58) (uuid "nc-bq-sdrv"))
-  (no_connect (at 257.81 78.74) (uuid "nc-bq-prog"))
-  (no_connect (at 257.81 81.28) (uuid "nc-bq-btst2"))
-  (no_connect (at 257.81 83.82) (uuid "nc-bq-batp"))
-  (no_connect (at 257.81 86.36) (uuid "nc-bq-ilim"))
-  (no_connect (at 257.81 88.9) (uuid "nc-bq-ts"))
-  (no_connect (at 87.63 180.34) (uuid "nc-xl-fb"))
-  (no_connect (at 87.63 185.42) (uuid "nc-xl-onoff"))
+  (symbol
+    (lib_id "power:PWR_FLAG")
+    (at 124.46 57.15 0)
+    (unit 1)
+    (exclude_from_sim no)
+    (in_bom no)
+    (on_board yes)
+    (dnp no)
+    (uuid "pwr-flag-vbus")
+    (property "Reference" "#FLG01"
+      (at 124.46 53.34 0)
+      (effects (font (size 1.27 1.27)) hide)
+    )
+    (property "Value" "PWR_FLAG"
+      (at 124.46 53.34 0)
+      (effects (font (size 1.27 1.27)))
+    )
+    (pin "1" (uuid "pin-flg-1"))
+    (instances
+      (project "sdr_transceiver"
+        (path "/sdr-root-uuid/power-mgmt-uuid-001" (reference "#FLG01") (unit 1))
+      )
+    )
+  )
 )
