File: sdr_kicad/usb_connectors.kicad_sch (KiCad schematic)
At the start: 6 parts

Commit message: Add missing schematic symbols and fix hierarchical connections
- Add USB-C receptacles (J1, J2) and USBLC6-2SC6 ESD ICs to usb_connectors
- Add FST3253 QSD, EC2-3SNU relays (K1-K5), SMA connector, 1N5711 diodes to rf_section
- Add missing sheet pins for proper hierarchical signal routing
- Remove invalid comment lines that broke KiCad parser
- Update power management to TPS25750D/BQ25798 architecture for 4S battery support
- ERC reduced from 89 to 82 violations (remaining are unwired connections)
Parts:
- added J1, J2: USB_C_Receptacle, Connector_USB:USB_C_Receptacle_HRO_TYPE-C-31-M-12, symbol Connector:USB_C_Receptacle_USB2.0
- added U10, U11: USBLC6-2SC6, Package_TO_SOT_SMD:SOT-23-6, symbol Power_Protection:USBLC6-2SC6
Other:
- note added: "USB-C Receptacle: 16-pin mid-mount type LCSC: C2765186 or similar Connections (TPS25750D Architecture): • VBUS → TPS25750D VBUS (direct) • CC1/CC2 → TPS25750D CC1/CC2 (direct) (NO external Rd resistors - TPS25750D has internal) • D+/D- → STM32 USB (via ESD) • SBU1/SBU2 → NC (reserved) • Shield → GND via 1M + 4.7nF Note: TPS25750D provides: • Integrated CC protection • Integrated VBUS switch (28V/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"
- note added: "USBLC6-2SC6: • SOT-23-6 package • ESD: ±15kV (air), ±8kV (contact) • Low capacitance: 2pF typ • LCSC: C7519 (Basic part) Pinout: 1: I/O1 (D+) 2: GND 3: I/O2 (D-) 4: I/O2 (D-) 5: VBUS (clamp ref) 6: I/O1 (D+) Note: CC lines protected by TPS25750D integrated ESD"
- note removed: "USB-C Receptacle: 16-pin mid-mount type LCSC: C2765186 or similar Connections: • VBUS → TCPP03 → BQ25713 • CC1/CC2 → TCPP03 → STM32 UCPD • D+/D- → STM32 USB (via ESD) • SBU1/SBU2 → NC (reserved) • Shield → GND via 1M + 4.7nF ESD Protection: USBLC6-2SC6 (C7519) - Basic Protects D+/D- lines"
- note removed: "USBLC6-2SC6: • SOT-23-6 package • ESD: ±15kV (air), ±8kV (contact) • Low capacitance: 2pF typ • LCSC: C7519 (Basic part) Pinout: 1: I/O1 (D+) 2: GND 3: I/O2 (D-) 4: I/O2 (D-) 5: VBUS (clamp ref) 6: I/O1 (D+)"

Commit message: Add Python KiCad helper library and JLCPCB component libraries
- Add kicad_lib: Python library for parsing, creating, and validating KiCad files
  - S-expression parser and writer for .kicad_sym and .kicad_sch files
  - Immutable dataclasses for symbols, schematics, pins, wires, etc.
  - SymbolBuilder with fluent API for programmatic symbol creation
  - ERC validation runner with configurable rules
  - Result type for explicit error handling

- Add custom_lib: JLCPCB component libraries downloaded via JLC2KiCadLib
  - 21 symbol definitions (.kicad_sym)
  - 19 footprints with 3D STEP models
  - Includes STM32G474, TPS25750D, BQ25798, Si5351A, FT4232HL, etc.

- Update CLAUDE.md with kicad_lib documentation and usage examples

- Update schematic sheets with embedded lib_symbols and wiring
Parts:
- J1, J2: symbol Connector:USB_C_Receptacle_USB2.0 -> USB-C-16PIN:TYPE-C_16PIN_2MD_073
- U10, U11: symbol Power_Protection:USBLC6-2SC6 -> USBLC6:USBLC6-2SC6
Changed lines of the file:
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@@
   )
   (symbol
-    (lib_id "Connector:USB_C_Receptacle_USB2.0")
+    (lib_id "USB-C-16PIN:TYPE-C_16PIN_2MD_073")
     (at 50.8 63.5 0)
     (unit 1)
@@
   )
   (symbol
-    (lib_id "Power_Protection:USBLC6-2SC6")
+    (lib_id "USBLC6:USBLC6-2SC6")
     (at 165.1 76.2 0)
     (unit 1)
@@
   )
   (symbol
-    (lib_id "Connector:USB_C_Receptacle_USB2.0")
+    (lib_id "USB-C-16PIN:TYPE-C_16PIN_2MD_073")
     (at 50.8 152.4 0)
     (unit 1)
@@
   )
   (symbol
-    (lib_id "Power_Protection:USBLC6-2SC6")
+    (lib_id "USBLC6:USBLC6-2SC6")
     (at 165.1 165.1 0)
     (unit 1)
@@
     (uuid "hlabel-usb2-dm")
   )
+  (wire (pts (xy 63.5 48.26) (xy 100 48.26)) (uuid "wire-j1-vbus-1"))
+  (wire (pts (xy 100 48.26) (xy 100 38.1)) (uuid "wire-j1-vbus-2"))
+  (wire (pts (xy 100 38.1) (xy 228.6 38.1)) (uuid "wire-j1-vbus-3"))
+  (wire (pts (xy 63.5 55.88) (xy 105 55.88)) (uuid "wire-j1-cc1-1"))
+  (wire (pts (xy 105 55.88) (xy 105 50.8)) (uuid "wire-j1-cc1-2"))
+  (wire (pts (xy 105 50.8) (xy 228.6 50.8)) (uuid "wire-j1-cc1-3"))
+  (wire (pts (xy 63.5 58.42) (xy 110 58.42)) (uuid "wire-j1-cc2-1"))
+  (wire (pts (xy 110 58.42) (xy 110 63.5)) (uuid "wire-j1-cc2-2"))
+  (wire (pts (xy 110 63.5) (xy 228.6 63.5)) (uuid "wire-j1-cc2-3"))
+  (wire (pts (xy 63.5 68.58) (xy 130 68.58)) (uuid "wire-j1-dp-1"))
+  (wire (pts (xy 130 68.58) (xy 130 71.12)) (uuid "wire-j1-dp-2"))
+  (wire (pts (xy 130 71.12) (xy 152.4 71.12)) (uuid "wire-j1-dp-3"))
+  (wire (pts (xy 63.5 73.66) (xy 125 73.66)) (uuid "wire-j1-dm-1"))
+  (wire (pts (xy 125 73.66) (xy 125 81.28)) (uuid "wire-j1-dm-2"))
+  (wire (pts (xy 125 81.28) (xy 152.4 81.28)) (uuid "wire-j1-dm-3"))
+  (wire (pts (xy 177.8 71.12) (xy 200 71.12)) (uuid "wire-esd1-dp-out-1"))
+  (wire (pts (xy 200 71.12) (xy 200 76.2)) (uuid "wire-esd1-dp-out-2"))
+  (wire (pts (xy 200 76.2) (xy 228.6 76.2)) (uuid "wire-esd1-dp-out-3"))
+  (wire (pts (xy 177.8 81.28) (xy 205 81.28)) (uuid "wire-esd1-dm-out-1"))
+  (wire (pts (xy 205 81.28) (xy 205 88.9)) (uuid "wire-esd1-dm-out-2"))
+  (wire (pts (xy 205 88.9) (xy 228.6 88.9)) (uuid "wire-esd1-dm-out-3"))
+  (wire (pts (xy 63.5 137.16) (xy 130 137.16)) (uuid "wire-j2-dp-1"))
+  (wire (pts (xy 130 137.16) (xy 130 160.02)) (uuid "wire-j2-dp-2"))
+  (wire (pts (xy 130 160.02) (xy 152.4 160.02)) (uuid "wire-j2-dp-3"))
+  (wire (pts (xy 63.5 142.24) (xy 125 142.24)) (uuid "wire-j2-dm-1"))
+  (wire (pts (xy 125 142.24) (xy 125 170.18)) (uuid "wire-j2-dm-2"))
+  (wire (pts (xy 125 170.18) (xy 152.4 170.18)) (uuid "wire-j2-dm-3"))
+  (wire (pts (xy 177.8 160.02) (xy 200 160.02)) (uuid "wire-esd2-dp-out-1"))
+  (wire (pts (xy 200 160.02) (xy 200 152.4)) (uuid "wire-esd2-dp-out-2"))
+  (wire (pts (xy 200 152.4) (xy 228.6 152.4)) (uuid "wire-esd2-dp-out-3"))
+  (wire (pts (xy 177.8 170.18) (xy 205 170.18)) (uuid "wire-esd2-dm-out-1"))
+  (wire (pts (xy 205 170.18) (xy 205 165.1)) (uuid "wire-esd2-dm-out-2"))
+  (wire (pts (xy 205 165.1) (xy 228.6 165.1)) (uuid "wire-esd2-dm-out-3"))
+  (wire (pts (xy 63.5 86.36) (xy 76.2 86.36)) (uuid "wire-j1-shield-1"))
+  (wire (pts (xy 76.2 86.36) (xy 76.2 106.68)) (uuid "wire-j1-shield-2"))
+  (wire (pts (xy 76.2 121.92) (xy 76.2 127)) (uuid "wire-j1-shield-3"))
+  (wire (pts (xy 76.2 127) (xy 88.9 127)) (uuid "wire-j1-shield-4"))
+  (wire (pts (xy 88.9 106.68) (xy 88.9 127)) (uuid "wire-j1-shield-5"))
+  (wire (pts (xy 63.5 175.26) (xy 76.2 175.26)) (uuid "wire-j2-shield-1"))
+  (wire (pts (xy 76.2 175.26) (xy 76.2 175.26)) (uuid "wire-j2-shield-2"))
+  (symbol
+    (lib_id "power:GND")
+    (at 76.2 127 0)
+    (unit 1)
+    (exclude_from_sim no)
+    (in_bom no)
+    (on_board yes)
+    (dnp no)
+    (uuid "pwr-gnd-usb1")
+    (property "Reference" "#PWR010"
+      (at 76.2 133.35 0)
+      (effects (font (size 1.27 1.27)) hide)
+    )
+    (property "Value" "GND"
+      (at 76.2 130.81 0)
+      (effects (font (size 1.27 1.27)))
+    )
+  )
+  (symbol
+    (lib_id "power:GND")
+    (at 76.2 195.58 0)
+    (unit 1)
+    (exclude_from_sim no)
+    (in_bom no)
+    (on_board yes)
+    (dnp no)
+    (uuid "pwr-gnd-usb2")
+    (property "Reference" "#PWR011"
+      (at 76.2 201.93 0)
+      (effects (font (size 1.27 1.27)) hide)
+    )
+    (property "Value" "GND"
+      (at 76.2 199.39 0)
+      (effects (font (size 1.27 1.27)))
+    )
+  )
+  (symbol
+    (lib_id "power:GND")
+    (at 165.1 88.9 0)
+    (unit 1)
+    (exclude_from_sim no)
+    (in_bom no)
+    (on_board yes)
+    (dnp no)
+    (uuid "pwr-gnd-esd1")
+    (property "Reference" "#PWR012"
+      (at 165.1 95.25 0)
+      (effects (font (size 1.27 1.27)) hide)
+    )
+    (property "Value" "GND"
+      (at 165.1 92.71 0)
+      (effects (font (size 1.27 1.27)))
+    )
+  )
+  (symbol
+    (lib_id "power:GND")
+    (at 165.1 177.8 0)
+    (unit 1)
+    (exclude_from_sim no)
+    (in_bom no)
+    (on_board yes)
+    (dnp no)
+    (uuid "pwr-gnd-esd2")
+    (property "Reference" "#PWR013"
+      (at 165.1 184.15 0)
+      (effects (font (size 1.27 1.27)) hide)
+    )
+    (property "Value" "GND"
+      (at 165.1 181.61 0)
+      (effects (font (size 1.27 1.27)))
+    )
+  )
+  (symbol
+    (lib_id "power:+5V")
+    (at 165.1 63.5 0)
+    (unit 1)
+    (exclude_from_sim no)
+    (in_bom no)
+    (on_board yes)
+    (dnp no)
+    (uuid "pwr-5v-esd1")
+    (property "Reference" "#PWR014"
+      (at 165.1 67.31 0)
+      (effects (font (size 1.27 1.27)) hide)
+    )
+    (property "Value" "+5V"
+      (at 165.1 59.69 0)
+      (effects (font (size 1.27 1.27)))
+    )
+  )
+  (symbol
+    (lib_id "power:+5V")
+    (at 165.1 152.4 0)
+    (unit 1)
+    (exclude_from_sim no)
+    (in_bom no)
+    (on_board yes)
+    (dnp no)
+    (uuid "pwr-5v-esd2")
+    (property "Reference" "#PWR015"
+      (at 165.1 156.21 0)
+      (effects (font (size 1.27 1.27)) hide)
+    )
+    (property "Value" "+5V"
+      (at 165.1 148.59 0)
+      (effects (font (size 1.27 1.27)))
+    )
+  )
+  (wire (pts (xy 101.6 157.48) (xy 101.6 175.26)) (uuid "wire-cc1-sink-gnd"))
+  (wire (pts (xy 114.3 157.48) (xy 114.3 175.26)) (uuid "wire-cc2-sink-gnd"))
+  (wire (pts (xy 101.6 175.26) (xy 114.3 175.26)) (uuid "wire-cc-sink-gnd-bus"))
+  (wire (pts (xy 114.3 175.26) (xy 130 175.26)) (uuid "wire-cc-sink-gnd-ext"))
+  (symbol
+    (lib_id "power:GND")
+    (at 130 175.26 0)
+    (unit 1)
+    (exclude_from_sim no)
+    (in_bom no)
+    (on_board yes)
+    (dnp no)
+    (uuid "pwr-gnd-cc-sink")
+    (property "Reference" "#PWR016"
+      (at 130 181.61 0)
+      (effects (font (size 1.27 1.27)) hide)
+    )
+    (property "Value" "GND"
+      (at 130 179.07 0)
+      (effects (font (size 1.27 1.27)))
+    )
+  )
+  (wire (pts (xy 63.5 144.78) (xy 101.6 144.78)) (uuid "wire-j2-cc1"))
+  (wire (pts (xy 101.6 144.78) (xy 101.6 157.48)) (uuid "wire-j2-cc1-sink"))
+  (wire (pts (xy 63.5 147.32) (xy 114.3 147.32)) (uuid "wire-j2-cc2"))
+  (wire (pts (xy 114.3 147.32) (xy 114.3 157.48)) (uuid "wire-j2-cc2-sink"))
+  (junction (at 101.6 175.26) (uuid "jct-cc-sink-1"))
+  (junction (at 114.3 175.26) (uuid "jct-cc-sink-2"))
+  (wire (pts (xy 76.2 190.5) (xy 76.2 195.58)) (uuid "wire-j2-shield-gnd"))
+  (wire (pts (xy 88.9 190.5) (xy 88.9 195.58)) (uuid "wire-j2-cap-gnd"))
+  (wire (pts (xy 76.2 195.58) (xy 88.9 195.58)) (uuid "wire-j2-shield-bus"))
+  (junction (at 76.2 195.58) (uuid "jct-gnd-usb2"))
 )

Commit message: schematic is still quite borked
Parts:
- C60, C61, R60, R61, R62, R63, U10, U11: JLC_Basic Yes -> (none)
Connections:
- net +5V: now also U10.5 (VBUS), U11.5 (VBUS)
- net CC1: now also J1.4 (CC1)
- net CC2: now also J1.10 (CC2)
- net GND: now also C60.2, C61.2, J1.1 (GND), J1.12 (GND), J2.1 (GND), J2.12 (GND), J2.5 (DN2), J2.7 (DN1), R60.2, R61.2, R62.2, R63.2, U10.2 (GND), U11.2 (GND), U11.3 (I/O2)
- net USB1_DM: now also U10.4 (I/O2)
- net USB1_DP: now also U10.6 (I/O1)
- net USB2_DM: now also U11.4 (I/O2)
- net USB2_DP: now also U11.6 (I/O1)
- net VBUS: now also J1.11 (VBUS), J1.2 (VBUS)
- net at C60.1: now also J1.13 (SHELL), J1.14 (SHELL), R60.1
- net at C61.1: now also J2.13 (SHELL), J2.14 (SHELL), R63.1
- net at J1.5 (DN2): now also J1.7 (DN1), U10.3 (I/O2)
- net at J1.6 (DP1): now also J1.8 (DP2), U10.1 (I/O1)
- net at J2.10 (CC2): now also R62.1
- net USB2_VBUS: now reaches J2.11 (VBUS)
- net USB2_VBUS: now also J2.2 (VBUS)
- net at J2.4 (CC1): now also R61.1
- net at J2.6 (DP1): now also J2.8 (DP2), U11.1 (I/O1)
- no-connect marks 0 -> 4
Other:
- note removed: "USB-C Receptacle: 16-pin mid-mount type LCSC: C2765186 or similar Connections (TPS25750D Architecture): • VBUS → TPS25750D VBUS (direct) • CC1/CC2 → TPS25750D CC1/CC2 (direct) (NO external Rd resistors - TPS25750D has internal) • D+/D- → STM32 USB (via ESD) • SBU1/SBU2 → NC (reserved) • Shield → GND via 1M + 4.7nF Note: TPS25750D provides: • Integrated CC protection • Integrated VBUS switch (28V/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"
- note removed: "USB-C Receptacle: 16-pin mid-mount type Same part as USB-C #1 Connections: • VBUS → 5V input for FT4232H • CC1/CC2 → 5.1k to GND (sink) • D+/D- → FT4232H USB • SBU1/SBU2 → NC No PD negotiation needed. Simple 5V sink configuration."
- note removed: "USBLC6-2SC6: • SOT-23-6 package • ESD: ±15kV (air), ±8kV (contact) • Low capacitance: 2pF typ • LCSC: C7519 (Basic part) Pinout: 1: I/O1 (D+) 2: GND 3: I/O2 (D-) 4: I/O2 (D-) 5: VBUS (clamp ref) 6: I/O1 (D+) Note: CC lines protected by TPS25750D integrated ESD"
- moved on the sheet: C60, C61, R60, R63

Commit message: add firmware and readme
Connections:
- net GND: now also C61.1, J2.13 (SHELL), J2.14 (SHELL), J2.3 (SBU2), R63.1
- net at C60.1, J1.13 (SHELL), J1.14 (SHELL)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: now also J1.5 (DN2), J1.7 (DN1), U10.3 (I/O2)
- no-connect marks 4 -> 12
Changed lines of the file:
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@@
   (junction (at 76.2 96.52) (diameter 0) (color 0 0 0 0) (uuid "jct-rc1-top"))
   (junction (at 76.2 185.42) (diameter 0) (color 0 0 0 0) (uuid "jct-rc2-top"))
+  ; J1 missing connections
+  ; GND pins
+  (wire (pts (xy 39.37 45.72) (xy 35 45.72)) (uuid "wire-j1-gnd1-1"))
+  (wire (pts (xy 35 45.72) (xy 35 35)) (uuid "wire-j1-gnd1-2"))
+  (wire (pts (xy 39.37 43.18) (xy 35 43.18)) (uuid "wire-j1-gnd12-1"))
+  (wire (pts (xy 35 43.18) (xy 35 35)) (uuid "wire-j1-gnd12-2"))
+  (junction (at 35 35) (uuid "jct-j1-gnd"))
+  (symbol
+    (lib_id "power:GND")
+    (at 35 35 0)
+    (unit 1)
+    (exclude_from_sim no)
+    (in_bom no)
+    (on_board yes)
+    (dnp no)
+    (uuid "pwr-gnd-j1")
+    (property "Reference" "#PWR017"
+      (at 35 41.35 0)
+      (effects (font (size 1.27 1.27)) hide)
+    )
+    (property "Value" "GND"
+      (at 35 38.81 0)
+      (effects (font (size 1.27 1.27)))
+    )
+  )
+  ; VBUS pin 11
+  (wire (pts (xy 39.37 50.80) (xy 30 50.80)) (uuid "wire-j1-vbus11-1"))
+  (wire (pts (xy 30 50.80) (xy 30 38.1)) (uuid "wire-j1-vbus11-2"))
+  (symbol
+    (lib_id "power:+5V")
+    (at 30 38.1 0)
+    (unit 1)
+    (exclude_from_sim no)
+    (in_bom no)
+    (on_board yes)
+    (dnp no)
+    (uuid "pwr-5v-j1-vbus11")
+    (property "Reference" "#PWR018"
+      (at 30 41.91 0)
+      (effects (font (size 1.27 1.27)) hide)
+    )
+    (property "Value" "+5V"
+      (at 30 34.29 0)
+      (effects (font (size 1.27 1.27)))
+    )
+  )
+  ; SHELL pin 13
+  (wire (pts (xy 60.96 83.82) (xy 76.2 83.82)) (uuid "wire-j1-shell13-1"))
+  (wire (pts (xy 76.2 83.82) (xy 76.2 86.36)) (uuid "wire-j1-shell13-2"))
+  ; No-connect flags for J1
+  (no_connect (at 39.37 53.34) (uuid "nc-j1-sbu2"))
+  (no_connect (at 39.37 60.96) (uuid "nc-j1-dn2"))
+  (no_connect (at 39.37 78.74) (uuid "nc-j1-dp2"))
+  (no_connect (at 39.37 81.28) (uuid "nc-j1-sbu1"))
+  ; J2 missing connections
+  ; GND pins
+  (wire (pts (xy 39.37 143.51) (xy 35 143.51)) (uuid "wire-j2-gnd1-1"))
+  (wire (pts (xy 35 143.51) (xy 35 124)) (uuid "wire-j2-gnd1-2"))
+  (wire (pts (xy 39.37 148.17) (xy 35 148.17)) (uuid "wire-j2-gnd12-1"))
+  (wire (pts (xy 35 148.17) (xy 35 124)) (uuid "wire-j2-gnd12-2"))
+  (junction (at 35 124) (uuid "jct-j2-gnd"))
+  (symbol
+    (lib_id "power:GND")
+    (at 35 124 0)
+    (unit 1)
+    (exclude_from_sim no)
+    (in_bom no)
+    (on_board yes)
+    (dnp no)
+    (uuid "pwr-gnd-j2")
+    (property "Reference" "#PWR019"
+      (at 35 130.35 0)
+      (effects (font (size 1.27 1.27)) hide)
+    )
+    (property "Value" "GND"
+      (at 35 127.81 0)
+      (effects (font (size 1.27 1.27)))
+    )
+  )
+  ; VBUS pins 2 and 11
+  (wire (pts (xy 39.37 116.84) (xy 30 116.84)) (uuid "wire-j2-vbus2-1"))
+  (wire (pts (xy 30 116.84) (xy 30 127)) (uuid "wire-j2-vbus2-2"))
+  (wire (pts (xy 39.37 162.56) (xy 30 162.56)) (uuid "wire-j2-vbus11-1"))
+  (wire (pts (xy 30 162.56) (xy 30 127)) (uuid "wire-j2-vbus11-2"))
+  (junction (at 30 127) (uuid "jct-j2-vbus"))
+  (symbol
+    (lib_id "power:+5V")
+    (at 30 127 0)
+    (unit 1)
+    (exclude_from_sim no)
+    (in_bom no)
+    (on_board yes)
+    (dnp no)
+    (uuid "pwr-5v-j2-vbus")
+    (property "Reference" "#PWR020"
+      (at 30 130.81 0)
+      (effects (font (size 1.27 1.27)) hide)
+    )
+    (property "Value" "+5V"
+      (at 30 123.19 0)
+      (effects (font (size 1.27 1.27)))
+    )
+  )
+  ; SHELL pin 13
+  (wire (pts (xy 60.96 172.72) (xy 76.2 172.72)) (uuid "wire-j2-shell13-1"))
+  (wire (pts (xy 76.2 172.72) (xy 76.2 175.26)) (uuid "wire-j2-shell13-2"))
+  ; No-connect flags for J2
+  (no_connect (at 39.37 134.62) (uuid "nc-j2-sbu2"))
+  (no_connect (at 39.37 139.7) (uuid "nc-j2-dn2"))
+  (no_connect (at 39.37 149.86) (uuid "nc-j2-dp2"))
+  (no_connect (at 39.37 154.94) (uuid "nc-j2-sbu1"))
 )
